File: viaems-mini/inputs.sch (KiCad schematic (older format))
At the start: 65 parts

Commit message: More updates
Parts:
- C42: renamed from C?; value C -> 1 uF
- gave numbers to parts that had none: 64
Connections:
- net SPR1-adc is gone; now on net SPR-adc: C25.1, D4.3, R81.1

Commit message: Progress
Parts:
- removed R91, R92, R93, R94: 220, symbol Device:R
- added C49: 10 uF, Capacitor_SMD:C_0805_2012Metric, symbol Device:C
- added C50, C54: 0.1 uF, Capacitor_SMD:C_0805_2012Metric, symbol Device:C
- added C56: 47 uF, Capacitor_SMD:C_0805_2012Metric, symbol Device:C
- added U11: LM2937-N, Package_TO_SOT_SMD:TO-263-3_TabPin2, symbol Regulator_Linear:LM2937xT
- C29: renamed from C18; footprint (none) -> Capacitor_SMD:C_0805_2012Metric
- C30: renamed from C19; footprint (none) -> Capacitor_SMD:C_0805_2012Metric
- C31: renamed from C20; footprint (none) -> Capacitor_SMD:C_0805_2012Metric
- C32: renamed from C21; footprint (none) -> Capacitor_SMD:C_0805_2012Metric
- C33: renamed from C22; footprint (none) -> Capacitor_SMD:C_0805_2012Metric
- C34: renamed from C23; footprint (none) -> Capacitor_SMD:C_0805_2012Metric
- C35: renamed from C24; footprint (none) -> Capacitor_SMD:C_0805_2012Metric
- C36: renamed from C25; footprint (none) -> Capacitor_SMD:C_0805_2012Metric
- C37: renamed from C26; footprint (none) -> Capacitor_SMD:C_0805_2012Metric
- C38: renamed from C27; footprint (none) -> Capacitor_SMD:C_0805_2012Metric
- C39: renamed from C28; value 0.47 uF -> 0.22 uF; footprint (none) -> Capacitor_SMD:C_0805_2012Metric
- C40: renamed from C29; footprint (none) -> Capacitor_SMD:C_0805_2012Metric
- C41: renamed from C30; footprint (none) -> Capacitor_SMD:C_0805_2012Metric
- C42: renamed from C31; footprint (none) -> Capacitor_SMD:C_0805_2012Metric
- C43: renamed from C32; footprint (none) -> Capacitor_SMD:C_0805_2012Metric
- C44: renamed from C33; footprint (none) -> Capacitor_SMD:C_0805_2012Metric
- C45: renamed from C34; footprint (none) -> Capacitor_SMD:C_0805_2012Metric
- C46: renamed from C35; footprint (none) -> Capacitor_SMD:C_0805_2012Metric
- C47: renamed from C36; footprint (none) -> Capacitor_SMD:C_0805_2012Metric
- C48: renamed from C37; footprint (none) -> Capacitor_SMD:C_0805_2012Metric
- C51: renamed from C38; footprint (none) -> Capacitor_SMD:C_0805_2012Metric
- C52: renamed from C39; footprint (none) -> Capacitor_SMD:C_0805_2012Metric
- C53: renamed from C40; footprint (none) -> Capacitor_SMD:C_0805_2012Metric
- C55: renamed from C41; footprint (none) -> Capacitor_SMD:C_0805_2012Metric
- C57: renamed from C42; footprint (none) -> Capacitor_SMD:C_0805_2012Metric
- R100: renamed from R103; footprint (none) -> Resistor_SMD:R_0805_2012Metric
- R101: renamed from R104; footprint (none) -> Resistor_SMD:R_0805_2012Metric
- R102: renamed from R105; footprint (none) -> Resistor_SMD:R_0805_2012Metric
- R103: renamed from R106; footprint (none) -> Resistor_SMD:R_0805_2012Metric
- R80: renamed from R79; footprint (none) -> Resistor_SMD:R_0805_2012Metric
- R81: renamed from R80; footprint (none) -> Resistor_SMD:R_0805_2012Metric
- R82: renamed from R81; footprint (none) -> Resistor_SMD:R_0805_2012Metric
- R83: renamed from R82; value 470 -> 220; footprint (none) -> Resistor_SMD:R_0805_2012Metric
- R84: renamed from R83; footprint (none) -> Resistor_SMD:R_0805_2012Metric
- R85: renamed from R84; footprint (none) -> Resistor_SMD:R_0805_2012Metric
- R86: renamed from R85; footprint (none) -> Resistor_SMD:R_0805_2012Metric
- R87: renamed from R86; footprint (none) -> Resistor_SMD:R_0805_2012Metric
- R88: renamed from R87; footprint (none) -> Resistor_SMD:R_0805_2012Metric
- R89: renamed from R88; footprint (none) -> Resistor_SMD:R_0805_2012Metric
- R90: renamed from R89; footprint (none) -> Resistor_SMD:R_0805_2012Metric
- R91: renamed from R90; footprint (none) -> Resistor_SMD:R_0805_2012Metric
- R92: renamed from R95; footprint (none) -> Resistor_SMD:R_0805_2012Metric
- R93: renamed from R96; footprint (none) -> Resistor_SMD:R_0805_2012Metric
- R94: renamed from R97; footprint (none) -> Resistor_SMD:R_0805_2012Metric
- R95: renamed from R98; footprint (none) -> Resistor_SMD:R_0805_2012Metric
- R96: renamed from R99; footprint (none) -> Resistor_SMD:R_0805_2012Metric
- R97: renamed from R100; footprint (none) -> Resistor_SMD:R_0805_2012Metric
- R98: renamed from R101; footprint (none) -> Resistor_SMD:R_0805_2012Metric
- R99: renamed from R102; footprint (none) -> Resistor_SMD:R_0805_2012Metric
- U10: footprint (none) -> Package_SO:QSOP-16_3.9x4.9mm_P0.635mm
- U7, U8: footprint (none) -> Sensor_Pressure:Freescale_98ARH99089A
- U9: footprint (none) -> Package_SO:SOIC-16_3.9x9.9mm_P1.27mm
Connections:
- net 5v_main: no longer C29.1, C30.1, C47.1, C48.1, D2.2, D3.2, D4.2, D5.2, D6.2, D7.2, R87.1, R88.1, U7.2 (Vcc), U8.2 (Vcc), U9.2 (REF), U9.3 (VDD)
- net CS: now also U9.1 (CS)
- net GND: now also C49.2, C50.2, C54.2, C56.2, U11.2 (GND)
- net MISO: now also U9.15 (DOUT)
- net MOSI: now also U9.14 (DIN)
- net SCLK: now also U9.16 (SCLK)
- new net 12v_switched: C49.1, C50.1, U11.1 (VI)
- new net 5v_adc: C29.1, C30.1, C47.1, C48.1, C54.1, C56.1, D2.2, D3.2, D4.2, D5.2, D6.2, D7.2, R87.1, R88.1, U11.3 (VO), U7.2 (Vcc), U8.2 (Vcc), U9.2 (REF), U9.3 (VDD)
Other:
- note added: "ADC Power"
- note added: "For MAP the ADC protection is reduced \nand a smaller capacitor to allow a larger bandwidth."
- moved on the sheet: C51, C52, C53, C55, C57, R100, R101, R102, R103, R92, R93, R94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

Commit message: more
Parts:
- C39: value 0.22 uF -> 0.47 uF
- C40: value 0.47 uF -> 0.22 uF
- C56: footprint Capacitor_SMD:C_0805_2012Metric -> Capacitor_SMD:C_1206_3216Metric; Digikey-Part (none) -> 478-9009-1-ND
- R83: value 220 -> 470
- R84: value 470 -> 220
Changed lines of the file:
@@
 P 2600 5550
 F 0 "R83" V 2500 5550 50  0000 C CNN
-F 1 "220" V 2600 5550 50  0000 C CNN
+F 1 "470" V 2600 5550 50  0000 C CNN
 F 2 "Resistor_SMD:R_0805_2012Metric" V 2530 5550 50  0001 C CNN
 F 3 "~" H 2600 5550 50  0001 C CNN
@@
 P 2850 5700
 F 0 "C39" H 2965 5746 50  0000 L CNN
-F 1 "0.22 uF" H 2965 5655 50  0000 L CNN
+F 1 "0.47 uF" H 2965 5655 50  0000 L CNN
 F 2 "Capacitor_SMD:C_0805_2012Metric" H 2888 5550 50  0001 C CNN
 F 3 "~" H 2850 5700 50  0001 C CNN
@@
 P 2600 6850
 F 0 "R84" V 2500 6850 50  0000 C CNN
-F 1 "470" V 2600 6850 50  0000 C CNN
+F 1 "220" V 2600 6850 50  0000 C CNN
 F 2 "Resistor_SMD:R_0805_2012Metric" V 2530 6850 50  0001 C CNN
 F 3 "~" H 2600 6850 50  0001 C CNN
@@
 P 2850 7000
 F 0 "C40" H 2965 7046 50  0000 L CNN
-F 1 "0.47 uF" H 2965 6955 50  0000 L CNN
+F 1 "0.22 uF" H 2965 6955 50  0000 L CNN
 F 2 "Capacitor_SMD:C_0805_2012Metric" H 2888 6850 50  0001 C CNN
 F 3 "~" H 2850 7000 50  0001 C CNN
@@
 	1    0    0    -1
 $EndComp
-Text Notes 1950 5250 0    50   ~ 0
+Text Notes 1800 6350 0    50   ~ 0
 For MAP the ADC protection is reduced \nand a smaller capacitor to allow a larger bandwidth.
 $Comp
@@
 F 0 "C56" H 9115 5696 50  0000 L CNN
 F 1 "47 uF" H 9115 5605 50  0000 L CNN
-F 2 "Capacitor_SMD:C_0805_2012Metric" H 9038 5500 50  0001 C CNN
+F 2 "Capacitor_SMD:C_1206_3216Metric" H 9038 5500 50  0001 C CNN
 F 3 "~" H 9000 5650 50  0001 C CNN
+F 4 "478-9009-1-ND" H 9000 5650 50  0001 C CNN "Digikey-Part"
 	1    9000 5650
 	1    0    0    -1

Commit message: more
Parts:
- R102, R103: footprint Resistor_SMD:R_0805_2012Metric -> Resistor_THT:R_Axial_DIN0204_L3.6mm_D1.6mm_P2.54mm_Vertical
- U10: symbol viaems:MAX9926UAEE+ -> viaems-mini-rescue:MAX9926UAEE+-viaems
- U7, U8: symbol Sensor_Pressure:MPXA6115A -> viaems-mini-rescue:MPXA6115A-Sensor_Pressure
- U9: symbol viaems:AD7888 -> viaems-mini-rescue:AD7888-viaems
Changed lines of the file:
@@
 EESchema Schematic File Version 4
-LIBS:viaems-mini-cache
-EELAYER 26 0
+EELAYER 30 0
 EELAYER END
 $Descr A4 11693 8268
@@
 IAT-adc
 $Comp
-L Sensor_Pressure:MPXA6115A U7
+L viaems-mini-rescue:MPXA6115A-Sensor_Pressure U7
 U 1 1 5E102466
 P 1750 5550
@@
 $EndComp
 $Comp
-L Sensor_Pressure:MPXA6115A U8
+L viaems-mini-rescue:MPXA6115A-Sensor_Pressure U8
 U 1 1 5E1131E0
 P 1750 6850
@@
 $EndComp
 $Comp
-L viaems:AD7888 U9
+L viaems-mini-rescue:AD7888-viaems U9
 U 1 1 5E115076
 P 4800 6250
@@
 Connection ~ 7700 1450
 $Comp
-L viaems:MAX9926UAEE+ U10
+L viaems-mini-rescue:MAX9926UAEE+-viaems U10
 U 1 1 5E13EA4E
 P 7200 2800
@@
 F 0 "R103" H 8770 3346 50  0000 L CNN
 F 1 "330" V 8700 3250 50  0000 L CNN
-F 2 "Resistor_SMD:R_0805_2012Metric" V 8630 3300 50  0001 C CNN
+F 2 "Resistor_THT:R_Axial_DIN0204_L3.6mm_D1.6mm_P2.54mm_Vertical" V 8630 3300 50  0001 C CNN
 F 3 "~" H 8700 3300 50  0001 C CNN
 	1    8700 3300
@@
 F 0 "R102" H 8770 2246 50  0000 L CNN
 F 1 "330" V 8700 2150 50  0000 L CNN
-F 2 "Resistor_SMD:R_0805_2012Metric" V 8630 2200 50  0001 C CNN
+F 2 "Resistor_THT:R_Axial_DIN0204_L3.6mm_D1.6mm_P2.54mm_Vertical" V 8630 2200 50  0001 C CNN
 F 3 "~" H 8700 2200 50  0001 C CNN
 	1    8700 2200
