File: viaems-mini/outputs.sch (KiCad schematic (older format))
At the start: 64 parts

Commit message: More updates
Parts:
- added C16: 0.1 uF, symbol Device:C
- added C17: 1 uF, symbol Device:C
- added Q3, Q4, Q7, Q8: VNL5090S5-E, symbol viaems:VNL5090S5-E
- added R16, R18, R23, R24, R32, R34, R36, R41, R43, R46, R49, R50: 1k, symbol Device:R
- added R17, R19, R31, R33, R35, R42, R44, R45: 100k, symbol Device:R
- added R51, R52, R53, R54: 150, symbol Device:R
- added U6: MIC4469, symbol viaems:MIC4469
- gave numbers to parts that had none: 64
Connections:
- net 5v_main: now also R23.1, R24.1, R49.1, R50.1
- net GND: now also C16.2, C17.2, R17.2, R19.2, R31.2, R33.2, R35.2, R42.2, R44.2, R45.2, U6.10 (4B), U6.2 (1B), U6.4 (2B), U6.6 (3B)
- net INJ-GND: now also Q3.6 (SOURCE), Q3.7 (SOURCE), Q4.6 (SOURCE), Q4.7 (SOURCE), Q7.6 (SOURCE), Q7.7 (SOURCE), Q8.6 (SOURCE), Q8.7 (SOURCE)
- net at C14.1, C15.1, JP2.2: now also C16.1, C17.1
- new net: R31.1, R32.2, U6.1 (1A)
- new net: R54.2, U6.11 (4Y)
- new net: R53.2, U6.12 (3Y)
- new net: R52.2, U6.13 (2Y)
- new net: R51.2, U6.14 (1Y)
- new net: R33.1, R34.2, U6.3 (2A)
- new net: R35.1, R36.2, U6.5 (3A)
- new net: R45.1, R46.2, U6.9 (4A)
- new net: Q4.1 (SUPPLY), R24.2
- new net: Q4.2 (INPUT), R18.1, R19.1
- new net: Q8.1 (SUPPLY), R50.2
- new net: Q8.2 (INPUT), R43.1, R44.1
- new net: Q3.1 (SUPPLY), R23.2
- new net: Q3.2 (INPUT), R16.1, R17.1
- new net: Q7.1 (SUPPLY), R49.2
- new net: Q7.2 (INPUT), R41.1, R42.1
- new net IG5: R32.1
- new net IG5-out: R51.1
- new net IG6: R34.1
- new net IG6-out: R52.1
- new net IG7: R36.1
- new net IG7-out: R53.1
- new net IG8: R46.1
- new net IG8-out: R54.1
- new net INJ5: R16.2
- new net INJ5-out: Q3.5 (DRAIN), Q3.8 (DRAIN)
- new net INJ6: R18.2
- new net INJ6-out: Q4.5 (DRAIN), Q4.8 (DRAIN)
- new net INJ7: R41.2
- new net INJ7-out: Q7.5 (DRAIN), Q7.8 (DRAIN)
- new net INJ8: R43.2
- new net INJ8-out: Q8.5 (DRAIN), Q8.8 (DRAIN)
- no-connect marks 12 -> 16
Other:
- moved on the sheet: C14, C15, JP2, Q1, Q2, Q5, Q6, R10, R11, R12, R13, R14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

Commit message: Progress
Parts:
- C25: renamed from C14; footprint (none) -> Capacitor_SMD:C_0805_2012Metric
- C26: renamed from C15; footprint (none) -> Capacitor_SMD:C_0805_2012Metric
- C27: renamed from C16; footprint (none) -> Capacitor_SMD:C_0805_2012Metric
- C28: renamed from C17; footprint (none) -> Capacitor_SMD:C_0805_2012Metric
- JP2: footprint (none) -> Connector_PinHeader_2.54mm:PinHeader_1x03_P2.54mm_Vertical
- Q1, Q10, Q11, Q12, Q13, Q14, Q15, Q16, Q2, Q3, Q4, Q5, Q6, Q7, Q8, Q9: footprint (none) -> Package_SO:SO-8_5.3x6.2mm_P1.27mm
- R10: renamed from R9; footprint (none) -> Resistor_SMD:R_0805_2012Metric
- R11: renamed from R10; footprint (none) -> Resistor_SMD:R_0805_2012Metric
- R12: renamed from R11; footprint (none) -> Resistor_SMD:R_0805_2012Metric
- R13: renamed from R12; footprint (none) -> Resistor_SMD:R_0805_2012Metric
- R14: renamed from R13; footprint (none) -> Resistor_SMD:R_0805_2012Metric
- R15: renamed from R14; footprint (none) -> Resistor_SMD:R_0805_2012Metric
- R16: renamed from R15; footprint (none) -> Resistor_SMD:R_0805_2012Metric
- R17: renamed from R16; footprint (none) -> Resistor_SMD:R_0805_2012Metric
- R18: renamed from R17; footprint (none) -> Resistor_SMD:R_0805_2012Metric
- R19: renamed from R18; footprint (none) -> Resistor_SMD:R_0805_2012Metric
- R20: renamed from R19; footprint (none) -> Resistor_SMD:R_0805_2012Metric
- R21: renamed from R20; footprint (none) -> Resistor_SMD:R_0805_2012Metric
- R22: renamed from R21; footprint (none) -> Resistor_SMD:R_0805_2012Metric
- R23: renamed from R22; footprint (none) -> Resistor_SMD:R_0805_2012Metric
- R24: renamed from R23; footprint (none) -> Resistor_SMD:R_0805_2012Metric
- R25: renamed from R24; footprint (none) -> Resistor_SMD:R_0805_2012Metric
- R26: renamed from R25; footprint (none) -> Resistor_SMD:R_0805_2012Metric
- R27: renamed from R26; footprint (none) -> Resistor_SMD:R_0805_2012Metric
- R28: renamed from R27; footprint (none) -> Resistor_SMD:R_0805_2012Metric
- R29: renamed from R28; footprint (none) -> Resistor_SMD:R_0805_2012Metric
- R30: renamed from R29; footprint (none) -> Resistor_SMD:R_0805_2012Metric
- R31: renamed from R30; footprint (none) -> Resistor_SMD:R_0805_2012Metric
- R32: renamed from R31; footprint (none) -> Resistor_SMD:R_0805_2012Metric
- R33: renamed from R32; footprint (none) -> Resistor_SMD:R_0805_2012Metric
- R34: renamed from R33; footprint (none) -> Resistor_SMD:R_0805_2012Metric
- R35: renamed from R34; footprint (none) -> Resistor_SMD:R_0805_2012Metric
- R36: renamed from R35; footprint (none) -> Resistor_SMD:R_0805_2012Metric
- R37: renamed from R36; footprint (none) -> Resistor_SMD:R_0805_2012Metric
- R38: renamed from R37; footprint (none) -> Resistor_SMD:R_0805_2012Metric
- R39: renamed from R38; footprint (none) -> Resistor_SMD:R_0805_2012Metric
- R40: renamed from R39; footprint (none) -> Resistor_SMD:R_0805_2012Metric
- R41: renamed from R40; footprint (none) -> Resistor_SMD:R_0805_2012Metric
- R42: renamed from R41; footprint (none) -> Resistor_SMD:R_0805_2012Metric
- R43: renamed from R42; footprint (none) -> Resistor_SMD:R_0805_2012Metric
- R44: renamed from R43; footprint (none) -> Resistor_SMD:R_0805_2012Metric
- R45: renamed from R44; footprint (none) -> Resistor_SMD:R_0805_2012Metric
- R46: renamed from R45; footprint (none) -> Resistor_SMD:R_0805_2012Metric
- R47: renamed from R46; footprint (none) -> Resistor_SMD:R_0805_2012Metric
- R48: renamed from R47; footprint (none) -> Resistor_SMD:R_0805_2012Metric
- R49: renamed from R48; footprint (none) -> Resistor_SMD:R_0805_2012Metric
- R50: renamed from R49; footprint (none) -> Resistor_SMD:R_0805_2012Metric
- R51: renamed from R50; footprint (none) -> Resistor_SMD:R_0805_2012Metric
- R52: renamed from R51; footprint (none) -> Resistor_SMD:R_0805_2012Metric
- R53: renamed from R52; footprint (none) -> Resistor_SMD:R_0805_2012Metric
- R54: renamed from R53; footprint (none) -> Resistor_SMD:R_0805_2012Metric
- R55: renamed from R54; footprint (none) -> Resistor_SMD:R_0805_2012Metric
- R56: renamed from R55; footprint (none) -> Resistor_SMD:R_0805_2012Metric
- R57: renamed from R56; footprint (none) -> Resistor_SMD:R_0805_2012Metric
- R58: renamed from R57; footprint (none) -> Resistor_SMD:R_0805_2012Metric
- R59: renamed from R58; footprint (none) -> Resistor_SMD:R_0805_2012Metric
- R60: renamed from R59; footprint (none) -> Resistor_SMD:R_0805_2012Metric
- R61: renamed from R60; footprint (none) -> Resistor_SMD:R_0805_2012Metric
- R62: renamed from R61; footprint (none) -> Resistor_SMD:R_0805_2012Metric
- R63: renamed from R62; footprint (none) -> Resistor_SMD:R_0805_2012Metric
- R64: renamed from R63; footprint (none) -> Resistor_SMD:R_0805_2012Metric
- R65: renamed from R64; footprint (none) -> Resistor_SMD:R_0805_2012Metric
- R66: renamed from R65; footprint (none) -> Resistor_SMD:R_0805_2012Metric
- R67: renamed from R66; footprint (none) -> Resistor_SMD:R_0805_2012Metric
- R68: renamed from R67; footprint (none) -> Resistor_SMD:R_0805_2012Metric
- R69: renamed from R68; footprint (none) -> Resistor_SMD:R_0805_2012Metric
- R70: renamed from R69; footprint (none) -> Resistor_SMD:R_0805_2012Metric
- R71: renamed from R70; footprint (none) -> Resistor_SMD:R_0805_2012Metric
- R72: renamed from R71; footprint (none) -> Resistor_SMD:R_0805_2012Metric
- R73: renamed from R72; footprint (none) -> Resistor_SMD:R_0805_2012Metric
- R74: renamed from R73; footprint (none) -> Resistor_SMD:R_0805_2012Metric
- R75: renamed from R74; footprint (none) -> Resistor_SMD:R_0805_2012Metric
- R76: renamed from R75; footprint (none) -> Resistor_SMD:R_0805_2012Metric
- R77: renamed from R76; footprint (none) -> Resistor_SMD:R_0805_2012Metric
- R78: renamed from R77; footprint (none) -> Resistor_SMD:R_0805_2012Metric
- R79: renamed from R78; footprint (none) -> Resistor_SMD:R_0805_2012Metric
- R8: renamed from R7; footprint (none) -> Resistor_SMD:R_0805_2012Metric
- R9: renamed from R8; footprint (none) -> Resistor_SMD:R_0805_2012Metric
- U5, U6: footprint (none) -> Package_SO:SOIC-16W_7.5x10.3mm_P1.27mm
Connections:
- net GND: now also U5.7 (GND), U5.8 (GND), U6.7 (GND), U6.8 (GND)
- net at U5.15 (Vs): now also C25.1, C26.1, C27.1, C28.1, JP2.2, U5.16 (Vs), U6.15 (Vs), U6.16 (Vs)

Commit message: more
Parts:
- renumbered Q13 to Q10, Q10 to Q11, Q14 to Q12, Q11 to Q13, Q15 to Q14, Q12 to Q15, Q5 to Q3, Q6 to Q4, Q3 to Q5, Q4 to Q6
Changed lines of the file:
@@
 NoConn ~ 1500 4850
 $Comp
-L viaems:VNL5090S5-E Q6
+L viaems:VNL5090S5-E Q4
 U 1 1 5E03E3CD
 P 4700 4700
-F 0 "Q6" H 4700 4965 50  0000 C CNN
+F 0 "Q4" H 4700 4965 50  0000 C CNN
 F 1 "VNL5090S5-E" H 4700 4874 50  0000 C CNN
 F 2 "Package_SO:SO-8_5.3x6.2mm_P1.27mm" H 4700 4700 50  0001 C CNN
@@
 NoConn ~ 1500 4000
 $Comp
-L viaems:VNL5090S5-E Q5
+L viaems:VNL5090S5-E Q3
 U 1 1 5E03F646
 P 4700 3850
-F 0 "Q5" H 4700 4115 50  0000 C CNN
+F 0 "Q3" H 4700 4115 50  0000 C CNN
 F 1 "VNL5090S5-E" H 4700 4024 50  0000 C CNN
 F 2 "Package_SO:SO-8_5.3x6.2mm_P1.27mm" H 4700 3850 50  0001 C CNN
@@
 $EndComp
 $Comp
-L viaems:VNL5090S5-E Q10
+L viaems:VNL5090S5-E Q11
 U 1 1 5E05223D
 P 7400 2800
-F 0 "Q10" H 7400 3065 50  0000 C CNN
+F 0 "Q11" H 7400 3065 50  0000 C CNN
 F 1 "VNL5090S5-E" H 7400 2974 50  0000 C CNN
 F 2 "Package_SO:SO-8_5.3x6.2mm_P1.27mm" H 7400 2800 50  0001 C CNN
@@
 $EndComp
 $Comp
-L viaems:VNL5090S5-E Q14
+L viaems:VNL5090S5-E Q12
 U 1 1 5E09C3B1
 P 9850 2550
-F 0 "Q14" H 9850 2815 50  0000 C CNN
+F 0 "Q12" H 9850 2815 50  0000 C CNN
 F 1 "VNL5090S5-E" H 9850 2724 50  0000 C CNN
 F 2 "Package_SO:SO-8_5.3x6.2mm_P1.27mm" H 9850 2550 50  0001 C CNN
@@
 $EndComp
 $Comp
-L viaems:VNL5090S5-E Q13
+L viaems:VNL5090S5-E Q10
 U 1 1 5E09C3E1
 P 9850 1350
-F 0 "Q13" H 9850 1615 50  0000 C CNN
+F 0 "Q10" H 9850 1615 50  0000 C CNN
 F 1 "VNL5090S5-E" H 9850 1524 50  0000 C CNN
 F 2 "Package_SO:SO-8_5.3x6.2mm_P1.27mm" H 9850 1350 50  0001 C CNN
@@
 $EndComp
 $Comp
-L viaems:VNL5090S5-E Q12
+L viaems:VNL5090S5-E Q15
 U 1 1 5E0A07BD
 P 7400 5600
-F 0 "Q12" H 7400 5865 50  0000 C CNN
+F 0 "Q15" H 7400 5865 50  0000 C CNN
 F 1 "VNL5090S5-E" H 7400 5774 50  0000 C CNN
 F 2 "Package_SO:SO-8_5.3x6.2mm_P1.27mm" H 7400 5600 50  0001 C CNN
@@
 $EndComp
 $Comp
-L viaems:VNL5090S5-E Q11
+L viaems:VNL5090S5-E Q13
 U 1 1 5E0A07ED
 P 7400 4100
-F 0 "Q11" H 7400 4365 50  0000 C CNN
+F 0 "Q13" H 7400 4365 50  0000 C CNN
 F 1 "VNL5090S5-E" H 7400 4274 50  0000 C CNN
 F 2 "Package_SO:SO-8_5.3x6.2mm_P1.27mm" H 7400 4100 50  0001 C CNN
@@
 $EndComp
 $Comp
-L viaems:VNL5090S5-E Q15
+L viaems:VNL5090S5-E Q14
 U 1 1 5E0A5F03
 P 9850 3800
-F 0 "Q15" H 9850 4065 50  0000 C CNN
+F 0 "Q14" H 9850 4065 50  0000 C CNN
 F 1 "VNL5090S5-E" H 9850 3974 50  0000 C CNN
 F 2 "Package_SO:SO-8_5.3x6.2mm_P1.27mm" H 9850 3800 50  0001 C CNN
@@
 	1400 5050 1400 5250
 $Comp
-L viaems:VNL5090S5-E Q4
+L viaems:VNL5090S5-E Q6
 U 1 1 5E1E8A14
 P 2050 6400
-F 0 "Q4" H 2050 6665 50  0000 C CNN
+F 0 "Q6" H 2050 6665 50  0000 C CNN
 F 1 "VNL5090S5-E" H 2050 6574 50  0000 C CNN
 F 2 "Package_SO:SO-8_5.3x6.2mm_P1.27mm" H 2050 6400 50  0001 C CNN
@@
 NoConn ~ 4150 6650
 $Comp
-L viaems:VNL5090S5-E Q3
+L viaems:VNL5090S5-E Q5
 U 1 1 5E1E8A72
 P 2050 5550
-F 0 "Q3" H 2050 5815 50  0000 C CNN
+F 0 "Q5" H 2050 5815 50  0000 C CNN
 F 1 "VNL5090S5-E" H 2050 5724 50  0000 C CNN
 F 2 "Package_SO:SO-8_5.3x6.2mm_P1.27mm" H 2050 5550 50  0001 C CNN

Commit message: more
Parts:
- Q1, Q10, Q11, Q12, Q13, Q14, Q15, Q16, Q2, Q3, Q4, Q5, Q6, Q7, Q8, Q9: symbol viaems:VNL5090S5-E -> viaems-mini-rescue:VNL5090S5-E-viaems
- U5, U6: symbol viaems:MIC4469 -> viaems-mini-rescue:MIC4469-viaems
Changed lines of the file:
@@
 EESchema Schematic File Version 4
-LIBS:viaems-mini-cache
-EELAYER 26 0
+EELAYER 30 0
 EELAYER END
 $Descr A4 11693 8268
@@
 $EndDescr
 $Comp
-L viaems:MIC4469 U5
+L viaems-mini-rescue:MIC4469-viaems U5
 U 1 1 5E011E3A
 P 2050 1750
@@
 Ignition
 $Comp
-L viaems:VNL5090S5-E Q2
+L viaems-mini-rescue:VNL5090S5-E-viaems Q2
 U 1 1 5E032387
 P 2050 4650
@@
 NoConn ~ 1500 4850
 $Comp
-L viaems:VNL5090S5-E Q4
+L viaems-mini-rescue:VNL5090S5-E-viaems Q4
 U 1 1 5E03E3CD
 P 4700 4700
@@
 NoConn ~ 4150 4900
 $Comp
-L viaems:VNL5090S5-E Q1
+L viaems-mini-rescue:VNL5090S5-E-viaems Q1
 U 1 1 5E03F616
 P 2050 3800
@@
 NoConn ~ 1500 4000
 $Comp
-L viaems:VNL5090S5-E Q3
+L viaems-mini-rescue:VNL5090S5-E-viaems Q3
 U 1 1 5E03F646
 P 4700 3850
@@
 $EndComp
 $Comp
-L viaems:VNL5090S5-E Q11
+L viaems-mini-rescue:VNL5090S5-E-viaems Q11
 U 1 1 5E05223D
 P 7400 2800
@@
 $EndComp
 $Comp
-L viaems:VNL5090S5-E Q9
+L viaems-mini-rescue:VNL5090S5-E-viaems Q9
 U 1 1 5E099227
 P 7400 1350
@@
 $EndComp
 $Comp
-L viaems:VNL5090S5-E Q12
+L viaems-mini-rescue:VNL5090S5-E-viaems Q12
 U 1 1 5E09C3B1
 P 9850 2550
@@
 $EndComp
 $Comp
-L viaems:VNL5090S5-E Q10
+L viaems-mini-rescue:VNL5090S5-E-viaems Q10
 U 1 1 5E09C3E1
 P 9850 1350
@@
 $EndComp
 $Comp
-L viaems:VNL5090S5-E Q15
+L viaems-mini-rescue:VNL5090S5-E-viaems Q15
 U 1 1 5E0A07BD
 P 7400 5600
@@
 $EndComp
 $Comp
-L viaems:VNL5090S5-E Q13
+L viaems-mini-rescue:VNL5090S5-E-viaems Q13
 U 1 1 5E0A07ED
 P 7400 4100
@@
 $EndComp
 $Comp
-L viaems:VNL5090S5-E Q16
+L viaems-mini-rescue:VNL5090S5-E-viaems Q16
 U 1 1 5E0A5ED3
 P 9850 5000
@@
 $EndComp
 $Comp
-L viaems:VNL5090S5-E Q14
+L viaems-mini-rescue:VNL5090S5-E-viaems Q14
 U 1 1 5E0A5F03
 P 9850 3800
@@
 	2100 1000 2100 1450
 $Comp
-L viaems:MIC4469 U6
+L viaems-mini-rescue:MIC4469-viaems U6
 U 1 1 5E0FBDEA
 P 4600 1750
@@
 	1400 5050 1400 5250
 $Comp
-L viaems:VNL5090S5-E Q6
+L viaems-mini-rescue:VNL5090S5-E-viaems Q6
 U 1 1 5E1E8A14
 P 2050 6400
@@
 NoConn ~ 1500 6600
 $Comp
-L viaems:VNL5090S5-E Q8
+L viaems-mini-rescue:VNL5090S5-E-viaems Q8
 U 1 1 5E1E8A43
 P 4700 6450
@@
 NoConn ~ 4150 6650
 $Comp
-L viaems:VNL5090S5-E Q5
+L viaems-mini-rescue:VNL5090S5-E-viaems Q5
 U 1 1 5E1E8A72
 P 2050 5550
@@
 NoConn ~ 1500 5750
 $Comp
-L viaems:VNL5090S5-E Q7
+L viaems-mini-rescue:VNL5090S5-E-viaems Q7
 U 1 1 5E1E8AA1
 P 4700 5600
