File: viaems-mini/viaems-mini.sch (KiCad schematic (older format))
At the start: 18 parts

Commit message: More updates
Parts:
- removed J?: Daughterboard, symbol Connector_Generic:Conn_02x08_Odd_Even
- removed J?: Trace, symbol Connector_Generic:Conn_02x06_Odd_Even
- removed J?: SPI_ADC, symbol Connector_Generic:Conn_01x05
- added C10, C13, C43, C44, C45, C46, C48, C8: 0.1 uF, symbol Device:C
- added C11, C12: 16 pF, symbol Device:C
- added C47: 4.7 uF, symbol Device:C
- added C49: 1 uF, symbol Device:C
- added C5, C6: 2.2 uF, symbol Device:C
- added J1: Primary, symbol Connector_Generic:Conn_02x06_Counter_Clockwise
- added J2: Power Drivers, symbol Connector_Generic:Conn_02x10_Odd_Even
- added J3: Ignition Trace, symbol Connector_Generic:Conn_01x09
- added J4: Injector Trace, symbol Connector_Generic:Conn_01x09
- added J5: Test Trigger, symbol Connector_Generic:Conn_01x02
- added J6: Trigger, symbol Connector_Generic:Conn_01x02
- added J7: Daughterboard, symbol Connector_Generic:Conn_02x07_Odd_Even
- added J8: Debug, Connector_PinHeader_1.27mm:PinHeader_2x05_P1.27mm_Vertical_SMD, symbol Connector:Conn_ARM_JTAG_SWD_10
- added JP1: Jumper, symbol Device:Jumper
- added R1: 1k, symbol Device:R
- added R2: 100k, symbol Device:R
- added R3: 120, symbol Device:R
- added R4: 220, symbol Device:R
- added U3: TJA1051T-3, Package_SO:SOIC-8_3.9x4.9mm_P1.27mm, symbol Interface_CAN_LIN:TJA1051T-3
- added Y1: Crystal, symbol Device:Crystal
- D1: renamed from D?; value D_Zener -> 5.6 V Zener
- F1: renamed from F?; value Polyfuse -> Polyfuse 200 mA
- gave numbers to parts that had none: 13
Connections:
- net labels added: ADC_CS, ADC_MISO, ADC_MOSI, ADC_SCLK, CANH, CANL, EXTRA4, IG1, IG2, IG3, IG4, IG5, IG6, IG7, IG8, INJ-GND, INJ1, INJ2, INJ3, INJ4, INJ5, INJ6, INJ7, INJ8, LSD-GND, LSD1, LSD2, LSD3, LSD4, LSD5, LSD6, LSD7, LSD8, NRST, PH0, PH1, SWDCLK
- net labels removed: OUT1, OUT2, OUT3, OUT4, OUT5, OUT6, OUT7, OUT8, SWCLK, TRIG1, TRIG2
- wire segments 156 -> 250
- no-connect marks 2 -> 4

Commit message: Progress
Parts:
- removed J5: Test Trigger, symbol Connector_Generic:Conn_01x02
- removed J6: Trigger, symbol Connector_Generic:Conn_01x02
- removed J7: Daughterboard, symbol Connector_Generic:Conn_02x07_Odd_Even
- removed U4: STM32F405RGTx, Package_QFP:LQFP-64_10x10mm_P0.5mm, symbol MCU_ST_STM32F4:STM32F405RGTx
- added C10, C6: 0.1 uF, Capacitor_SMD:C_0805_2012Metric, symbol Device:C
- added C11, C9: 1 uF, Capacitor_SMD:C_0805_2012Metric, symbol Device:C
- added J10: TEST, Connector_PinHeader_2.54mm:PinHeader_1x02_P2.54mm_Vertical, symbol Connector_Generic:Conn_01x02
- added J14: Micro_SD_Card, Connector_Card:microSD_HC_Wuerth_693072010801, symbol Connector:Micro_SD_Card
- added J5: GPIO58, Connector_PinHeader_2.54mm:PinHeader_1x04_P2.54mm_Vertical, symbol Connector_Generic:Conn_01x04
- added J6: SPI1, Connector_PinHeader_2.54mm:PinHeader_1x04_P2.54mm_Vertical, symbol Connector_Generic:Conn_01x04
- added J7: PORTC, Connector_PinHeader_2.54mm:PinHeader_1x08_P2.54mm_Vertical, symbol Connector_Generic:Conn_01x08
- added J8: PWM56, Connector_PinHeader_2.54mm:PinHeader_1x02_P2.54mm_Vertical, symbol Connector_Generic:Conn_01x02
- added J9: CAN2, Connector_PinHeader_2.54mm:PinHeader_1x02_P2.54mm_Vertical, symbol Connector_Generic:Conn_01x02
- added R4: 100k, Resistor_SMD:R_0805_2012Metric, symbol Device:R
- added U4: STM32F427VGTx, Package_QFP:LQFP-100_14x14mm_P0.5mm, symbol MCU_ST_STM32F4:STM32F427VGTx
- C1: renamed from C43; footprint (none) -> Capacitor_SMD:C_0805_2012Metric
- C12: renamed from C46; footprint (none) -> Capacitor_SMD:C_0805_2012Metric
- C13: renamed from C3; footprint (none) -> Capacitor_SMD:C_0805_2012Metric
- C14: renamed from C47; footprint (none) -> Capacitor_SMD:C_0805_2012Metric
- C15: renamed from C4; footprint (none) -> Capacitor_SMD:C_0805_2012Metric
- C16: renamed from C48; footprint (none) -> Capacitor_SMD:C_0805_2012Metric
- C17: renamed from C49; footprint (none) -> Capacitor_SMD:C_0805_2012Metric
- C18: renamed from C6; footprint (none) -> Capacitor_SMD:C_0805_2012Metric
- C19: renamed from C5; footprint (none) -> Capacitor_SMD:C_0805_2012Metric
- C2: renamed from C8; footprint (none) -> Capacitor_SMD:C_0805_2012Metric
- C20: renamed from C7; footprint (none) -> Capacitor_SMD:C_0805_2012Metric
- C21: renamed from C9; footprint (none) -> Capacitor_SMD:C_0805_2012Metric
- C22: renamed from C11; footprint (none) -> Capacitor_SMD:C_0805_2012Metric
- C23: renamed from C13; footprint (none) -> Capacitor_SMD:C_0805_2012Metric
- C24: renamed from C12; footprint (none) -> Capacitor_SMD:C_0805_2012Metric
- C3: renamed from C44; footprint (none) -> Capacitor_SMD:C_0805_2012Metric
- C4: renamed from C1; footprint (none) -> Capacitor_SMD:C_0805_2012Metric
- C5: renamed from C45; footprint (none) -> Capacitor_SMD:C_0805_2012Metric
- C7: renamed from C2; footprint (none) -> Capacitor_SMD:C_0805_2012Metric
- C8: renamed from C10; footprint (none) -> Capacitor_SMD:C_0805_2012Metric
- D1: footprint (none) -> Diode_SMD:D_0805_2012Metric
- F1: value Polyfuse 200 mA -> Polyfuse 100 mA; footprint (none) -> Fuse:Fuse_0805_2012Metric; Digikey-Part (none) -> 507-1810-2-ND
- J1: renamed from J2; footprint (none) -> Connector_PinHeader_2.54mm:PinHeader_2x10_P2.54mm_Vertical
- J11: renamed from J10; footprint (none) -> Connector_PinHeader_2.54mm:PinHeader_2x08_P2.54mm_Vertical
- J13: renamed from J9; footprint (none) -> Connector_USB:USB_Micro-B_Amphenol_10103594-0001LF_Horizontal
- J2: renamed from J1; footprint (none) -> Connector_PinHeader_2.54mm:PinHeader_2x06_P2.54mm_Vertical
- J3, J4: footprint (none) -> Connector_PinHeader_2.54mm:PinHeader_1x09_P2.54mm_Vertical
- JP1: value Jumper -> LOAD; footprint (none) -> Connector_PinHeader_2.54mm:PinHeader_1x02_P2.54mm_Vertical
- R1: renamed from R3; footprint (none) -> Resistor_SMD:R_0805_2012Metric
- R2: renamed from R1; footprint (none) -> Resistor_SMD:R_0805_2012Metric
- R3: renamed from R2; footprint (none) -> Resistor_SMD:R_0805_2012Metric
- R5, R6: footprint (none) -> Resistor_SMD:R_0805_2012Metric
- R7: renamed from R4; footprint (none) -> Resistor_SMD:R_0805_2012Metric
- U2: renamed from U1; value LM2940-N -> LM2937-N
- U3: renamed from U2; footprint (none) -> Package_TO_SOT_SMD:TO-263-2
- Y1: footprint (none) -> Crystal:Crystal_HC49-U_Vertical
- renumbered J8 to J12, U3 to U1
Connections:
- net 3v_main: now also C10.1, C11.1, C6.1, C9.1, J14.4 (VDD), U4.100 (VDD), U4.11 (VDD), U4.19 (VDD), U4.21 (VREF+), U4.22 (VDDA), U4.28 (VDD), U4.50 (VDD), U4.6 (VBAT), U4.75 (VDD)
- net 5v_main: no longer D1.1 (K), F1.2
- net CAN_RX: now also U4.95 (PB8)
- net CAN_TX: now also U4.96 (PB9)
- net GND: now also J13.5 (GND), J13.6 (Shield), C10.2, C11.2, C6.2, C9.2, J14.6 (VSS), J14.9 (SHIELD), R4.2, U4.10 (VSS), U4.20 (VSSA), U4.27 (VSS), U4.74 (VSS), U4.99 (VSS)
- net GPIO1: now also U4.55 (PD8)
- net GPIO2: now also U4.56 (PD9)
- net GPIO3: now also U4.57 (PD10)
- net GPIO4: now also U4.58 (PD11)
- net Inputs/DIG1-cpu: now also U4.25 (PA2)
- net Inputs/DIG2-cpu: now also U4.26 (PA3)
- net Inputs/TRIG1: now also U4.23 (PA0)
- net Inputs/TRIG2: now also U4.24 (PA1)
- net NRST: now also U4.14 (NRST)
- net Outputs/IG1: now also U4.97 (PE0)
- net Outputs/IG2: now also U4.98 (PE1)
- net Outputs/IG3: now also U4.1 (PE2)
- net Outputs/IG4: now also U4.2 (PE3)
- net Outputs/IG5: now also U4.3 (PE4)
- net Outputs/IG6: now also U4.4 (PE5)
- net Outputs/IG7: now also U4.5 (PE6)
- net Outputs/IG8: now also U4.38 (PE7)
- net Outputs/INJ1: now also U4.39 (PE8)
- net Outputs/INJ2: now also U4.40 (PE9)
- net Outputs/INJ3: now also U4.41 (PE10)
- net Outputs/INJ4: now also U4.42 (PE11)
- net Outputs/INJ5: now also U4.43 (PE12)
- net Outputs/INJ6: now also U4.44 (PE13)
- net Outputs/INJ7: now also U4.45 (PE14)
- net Outputs/INJ8: now also U4.46 (PE15)
- net PH0: now also U4.12 (PH0)
- net PH1: now also U4.13 (PH1)
- net PWM1: now also U4.67 (PA8)
- net PWM2: now also U4.69 (PA10)
- net SWDCLK: now also U4.76 (PA14)
- net SWDIO: now also U4.72 (PA13)
- net USB_DM: now also U4.70 (PA11)
- net USB_DP: now also U4.71 (PA12)
- net USB_VBUS: now also U4.68 (PA9)
- net at C19.1: now also U4.73 (VCAP_2)
- net at C18.1: now also U4.49 (VCAP_1)
- net at R2.1, R3.1: now also U4.94 (BOOT0)
- net PWM5: now reaches J12.6 (SWO/TDO)
- net PWM5: now also J8.1 (Pin_1), U4.89 (PB3)
- new net: J7.1 (Pin_1), U4.15 (PC0)
- new net: J7.2 (Pin_2), U4.16 (PC1)
- new net: J7.3 (Pin_3), U4.17 (PC2)
- new net: J7.4 (Pin_4), U4.18 (PC3)
- new net: J6.1 (Pin_1), U4.29 (PA4)
- new net: J6.2 (Pin_2), U4.30 (PA5)
- new net: J6.3 (Pin_3), U4.31 (PA6)
- new net: J6.4 (Pin_4), U4.32 (PA7)
- new net: J7.5 (Pin_5), U4.33 (PC4)
- new net: J7.6 (Pin_6), U4.34 (PC5)
- new net: R4.1, U4.37 (PB2)
- new net: J5.4 (Pin_4), U4.59 (PD12)
- new net: J5.3 (Pin_3), U4.60 (PD13)
- new net: J5.2 (Pin_2), U4.61 (PD14)
- new net: J5.1 (Pin_1), U4.62 (PD15)
- new net: J7.7 (Pin_7), U4.63 (PC6)
- new net: J7.8 (Pin_8), U4.64 (PC7)
- new net 5v_adc: D1.1 (K), F1.2
- new net CAN2_RX: J9.1 (Pin_1), U4.91 (PB5)
- new net CAN2_TX: J9.2 (Pin_2), U4.92 (PB6)
- new net Inputs/CS: U4.51 (PB12)
- new net Inputs/MISO: U4.53 (PB14)
- new net Inputs/MOSI: U4.54 (PB15)
- new net Inputs/SCLK: U4.52 (PB13)
- new net PWM3: U4.35 (PB0)
- new net PWM4: U4.36 (PB1)
- new net PWM6: J8.2 (Pin_2), U4.90 (PB4)
- new net SDIO_CK: J14.5 (CLK), U4.80 (PC12)
- new net SDIO_CMD: J14.3 (CMD), U4.83 (PD2)
- new net SDIO_D0: J14.7 (DAT0), U4.65 (PC8)
- new net SDIO_D1: J14.8 (DAT1), U4.66 (PC9)
- new net SDIO_D2: J14.1 (DAT2), U4.78 (PC10)
- new net SDIO_D3: J14.2 (DAT3/CD), U4.79 (PC11)
- new net TEST1: J10.1 (Pin_1), U4.47 (PB10)
- new net TEST2: J10.2 (Pin_2), U4.48 (PB11)
- no-connect marks 4 -> 14
Other:
- note added: "CAN"
- moved on the sheet: C1, C12, C14, C16, C17, C18, C19, C2, C22, C23, C24, C3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

Commit message: more
Parts:
- removed J1: Power Drivers, Connector_PinHeader_2.54mm:PinHeader_2x10_P2.54mm_Vertical, symbol Connector_Generic:Conn_02x10_Odd_Even
- removed J13: USB_B_Micro, Connector_USB:USB_Micro-B_Amphenol_10103594-0001LF_Horizontal, symbol Connector:USB_B_Micro
- removed J14: Micro_SD_Card, Connector_Card:microSD_HC_Wuerth_693072010801, symbol Connector:Micro_SD_Card
- added J14: USB_B, Connector_USB:USB_B_OST_USB-B1HSxx_Horizontal, symbol Connector:USB_B
- added J15: Micro SD, Connector_Card:microSD_HC_Hirose_DM3D-SF, symbol Connector:Micro_SD_Card_Det_Hirose_DM3AT
- added J2: Injectors, Connector_PinHeader_2.54mm:PinHeader_1x10_P2.54mm_Vertical, symbol Connector_Generic:Conn_01x10
- added J3: LSD, Connector_PinHeader_2.54mm:PinHeader_1x10_P2.54mm_Vertical, symbol Connector_Generic:Conn_01x10
- C15: footprint Capacitor_SMD:C_0805_2012Metric -> Capacitor_SMD:C_1206_3216Metric; Digikey-Part (none) -> 478-9009-1-ND
- J13: renamed from J12; Digikey-Part (none) -> SAM9438-ND
- U2: footprint Package_TO_SOT_THT:TO-220-3_Vertical -> Package_TO_SOT_THT:TO-220-3_Horizontal_TabDown
- renumbered J2 to J1, J9 to J10, J10 to J11, J11 to J12, J3 to J4, J4 to J5, J5 to J6, J6 to J7, J7 to J8, J8 to J9
Connections:
- net 3v_main: now also J15.4 (VDD)
- net GND: now also J14.4 (GND), J14.5 (Shield), J15.11 (SHIELD), J15.6 (VSS)
- net INJ-GND: now also J2.5 (Pin_5), J2.6 (Pin_6)
- net INJ1: now also J2.1 (Pin_1)
- net INJ2: now also J2.2 (Pin_2)
- net INJ3: now also J2.3 (Pin_3)
- net INJ4: now also J2.4 (Pin_4)
- net INJ5: now also J2.7 (Pin_7)
- net INJ6: now also J2.8 (Pin_8)
- net INJ7: now also J2.9 (Pin_9)
- net INJ8: now also J2.10 (Pin_10)
- net LSD-GND: now also J3.5 (Pin_5), J3.6 (Pin_6)
- net LSD1: now also J3.1 (Pin_1)
- net LSD2: now also J3.2 (Pin_2)
- net LSD3: now also J3.3 (Pin_3)
- net LSD4: now also J3.4 (Pin_4)
- net LSD5: now also J3.7 (Pin_7)
- net LSD6: now also J3.8 (Pin_8)
- net LSD7: now also J3.9 (Pin_9)
- net LSD8: now also J3.10 (Pin_10)
- net SDIO_CK: now also J15.5 (CLK)
- net SDIO_CMD: now also J15.3 (CMD)
- net SDIO_D0: now also J15.7 (DAT0)
- net SDIO_D1: now also J15.8 (DAT1)
- net SDIO_D2: now also J15.1 (DAT2)
- net SDIO_D3: now also J15.2 (DAT3/CD)
- net USB_DM: now also J14.2 (D-)
- net USB_DP: now also J14.3 (D+)
- net at R5.2: now also J14.1 (VBUS)
- no-connect marks 14 -> 15
Other:
- moved on the sheet: C23, J13

Commit message: more
Parts:
- D1: footprint Diode_SMD:D_0805_2012Metric -> Diode_THT:D_DO-41_SOD81_P2.54mm_Vertical_AnodeUp
- F1: Digikey-Part 507-1810-2-ND -> 283-PTS080524V010CT-ND
- J1: symbol Connector_Generic:Conn_02x06_Counter_Clockwise -> Connector_Generic:Conn_02x06_Odd_Even
- J13: symbol Connector:Conn_ARM_JTAG_SWD_10 -> viaems-mini-rescue:Conn_ARM_JTAG_SWD_10-Connector
- J14: symbol Connector:USB_B -> viaems-mini-rescue:USB_B-Connector
- J15: symbol Connector:Micro_SD_Card_Det_Hirose_DM3AT -> viaems-mini-rescue:Micro_SD_Card_Det_Hirose_DM3AT-Connector
- U3: symbol viaems:LM2940 -> viaems-mini-rescue:LM2940-viaems
Connections:
- net 12v_switched: now also J1.2 (Pin_2); no longer J1.12 (Pin_12)
- net CANH: now also J1.12 (Pin_12); no longer J1.11 (Pin_11)
- net CANL: now also J1.11 (Pin_11); no longer J1.2 (Pin_2)
- net IG2: now also J1.5 (Pin_5); no longer J1.4 (Pin_4)
- net IG3: now also J1.7 (Pin_7); no longer J1.5 (Pin_5)
- net IG4: now also J1.9 (Pin_9); no longer J1.6 (Pin_6)
- net IG5: now also J1.4 (Pin_4); no longer J1.10 (Pin_10)
- net IG6: now also J1.6 (Pin_6); no longer J1.9 (Pin_9)
- net IG8: now also J1.10 (Pin_10); no longer J1.7 (Pin_7)
- net Inputs/BRV renamed SPR
- net Inputs/CLT renamed IN1+
- net Inputs/DIG1 renamed IN2-
- net Inputs/DIG2 renamed DIG1
- net Inputs/EGO renamed CLT
- net Inputs/IAT renamed IN2+
- net Inputs/IN1+ renamed TPS
- net Inputs/IN1- renamed BRV
- net Inputs/IN2+ renamed IAT
- net Inputs/IN2- renamed IN1-
- net Inputs/SPR renamed DIG2
- net Inputs/TPS renamed EGO
Changed lines of the file:
@@
 EESchema Schematic File Version 4
-LIBS:viaems-mini-cache
-EELAYER 26 0
+EELAYER 30 0
 EELAYER END
 $Descr A4 11693 8268
@@
 	0    1    1    0
 $EndComp
-Wire Wire Line
-	8900 3600 9850 3600
-Wire Wire Line
-	9850 3600 9850 3050
-Wire Wire Line
-	9750 3050 9750 3500
-Wire Wire Line
-	9750 3500 8900 3500
-Wire Wire Line
-	8900 3400 9650 3400
-Wire Wire Line
-	9650 3400 9650 3050
-Wire Wire Line
-	9550 3050 9550 3300
-Wire Wire Line
-	9550 3300 8900 3300
-Wire Wire Line
-	8900 3200 9450 3200
-Wire Wire Line
-	9450 3200 9450 3050
-Wire Wire Line
-	9350 3050 9350 3100
-Wire Wire Line
-	9350 3100 8900 3100
-Wire Wire Line
-	9350 2550 8900 2550
-Wire Wire Line
-	8900 2450 9450 2450
-Wire Wire Line
-	9450 2450 9450 2550
-Wire Wire Line
-	9550 2550 9550 2200
-Wire Wire Line
-	9550 2200 8900 2200
-Wire Wire Line
-	8900 2100 9650 2100
-Wire Wire Line
-	9650 2100 9650 2550
-Wire Wire Line
-	9750 2550 9750 2000
-Wire Wire Line
-	9750 2000 8900 2000
-Wire Wire Line
-	8900 1900 9850 1900
-Wire Wire Line
-	9850 1900 9850 2550
 $Comp
 L power:GND #PWR027
@@
 	9950 3200 10050 3200
 $Comp
-L viaems:LM2940 U3
+L viaems-mini-rescue:LM2940-viaems U3
 U 1 1 5E1B6337
 P 5100 1000
@@
 $EndComp
 $Comp
-L Connector:Conn_ARM_JTAG_SWD_10 J13
+L viaems-mini-rescue:Conn_ARM_JTAG_SWD_10-Connector J13
 U 1 1 5E377F32
 P 9000 5750
@@
 IG8
 $Comp
-L Connector_Generic:Conn_02x06_Counter_Clockwise J1
+L Connector_Generic:Conn_02x06_Odd_Even J1
 U 1 1 5E5F28AF
 P 1150 3850
@@
 12v_switched
 Wire Wire Line
-	950  3650 950  3500
-Wire Wire Line
 	950  3500 750  3500
+Text Label 950  3750 2    50   ~ 0
+IG1
 Text Label 950  3850 2    50   ~ 0
-IG1
+IG2
 Text Label 950  3950 2    50   ~ 0
-IG2
+IG3
 Text Label 950  4050 2    50   ~ 0
-IG3
+IG4
+Text Label 1450 3750 0    50   ~ 0
+IG5
+Text Label 1450 3850 0    50   ~ 0
+IG6
+Text Label 1450 3950 0    50   ~ 0
+IG7
+Text Label 1450 4050 0    50   ~ 0
+IG8
 Text Label 950  4150 2    50   ~ 0
-IG4
-Text Label 1450 3850 0    50   ~ 0
-IG5
-Text Label 1450 3950 0    50   ~ 0
-IG6
-Text Label 1450 4050 0    50   ~ 0
-IG7
+CANL
 Text Label 1450 4150 0    50   ~ 0
-IG8
-Text Label 950  3750 2    50   ~ 0
-CANL
-Text Label 1450 3750 0    50   ~ 0
 CANH
 Text Label 1050 4750 2    50   ~ 0
@@
 F 0 "D1" V 6854 1179 50  0000 L CNN
 F 1 "5.6 V Zener" V 6945 1179 50  0000 L CNN
-F 2 "Diode_SMD:D_0805_2012Metric" H 6900 1100 50  0001 C CNN
-F 3 "~" H 6900 1100 50  0001 C CNN
+F 2 "Diode_THT:D_DO-41_SOD81_P2.54mm_Vertical_AnodeUp" H 6900 1100 50  0001 C CNN
+F 3 "1N4734A-T50ACT-ND" H 6900 1100 50  0001 C CNN
 	1    6900 1100
 	0    1    1    0
@@
 F 2 "Fuse:Fuse_0805_2012Metric" H 7250 750 50  0001 L CNN
 F 3 "~" H 7200 950 50  0001 C CNN
-F 4 "507-1810-2-ND" V 7200 950 50  0001 C CNN "Digikey-Part"
+F 4 "283-PTS080524V010CT-ND" V 7200 950 50  0001 C CNN "Digikey-Part"
 	1    7200 950
 	0    1    1    0
@@
 Connection ~ 9950 1450
 $Comp
-L Connector:USB_B J14
+L viaems-mini-rescue:USB_B-Connector J14
 U 1 1 5F7830FA
 P 9950 1050
@@
 $EndComp
 $Comp
-L Connector:Micro_SD_Card_Det_Hirose_DM3AT J15
+L viaems-mini-rescue:Micro_SD_Card_Det_Hirose_DM3AT-Connector J15
 U 1 1 5F825F7B
 P 10200 4450
@@
 NoConn ~ 9300 4850
 NoConn ~ 9300 4950
+Wire Wire Line
+	950  3500 950  3650
+Text Label 8900 3100 0    50   ~ 0
+SPR
+Text Label 8900 3200 0    50   ~ 0
+IAT
+Text Label 8900 3300 0    50   ~ 0
+CLT
+Text Label 8900 3400 0    50   ~ 0
+BRV
+Text Label 8900 3500 0    50   ~ 0
+EGO
+Text Label 8900 3600 0    50   ~ 0
+TPS
+Text Label 8900 2450 0    50   ~ 0
+DIG1
+Text Label 8900 2550 0    50   ~ 0
+DIG2
+Text Label 8900 1900 0    50   ~ 0
+IN1+
+Text Label 8900 2000 0    50   ~ 0
+IN1-
+Text Label 8900 2100 0    50   ~ 0
+IN2+
+Text Label 8900 2200 0    50   ~ 0
+IN2-
+Text Label 9350 2550 1    50   ~ 0
+DIG1
+Text Label 9350 3050 3    50   ~ 0
+DIG2
+Text Label 9450 2550 1    50   ~ 0
+IN2-
+Text Label 9450 3050 3    50   ~ 0
+IN2+
+Text Label 9550 2550 1    50   ~ 0
+IN1-
+Text Label 9550 3050 3    50   ~ 0
+IN1+
+Text Label 9850 2550 1    50   ~ 0
+TPS
+Text Label 9850 3050 3    50   ~ 0
+EGO
+Text Label 9750 2550 1    50   ~ 0
+BRV
+Text Label 9750 3050 3    50   ~ 0
+CLT
+Text Label 9650 2550 1    50   ~ 0
+IAT
+Text Label 9650 3050 3    50   ~ 0
+SPR
 $EndSCHEMATC
