File: proto-s323k44/proto-s32k344.kicad_sch (KiCad schematic)
At the start: 47 parts, among them J1 USB_C_Receptacle_USB2.0, J2 USB_GPIO, U1 LM2940, U2 TL760, U3 LF15_TO252, U4 M24C02-WMN, U5 XR21V1410, U6 TJA1101B

Commit message: more work on s32k3
Parts:
- removed C1, C3, C4, C5, C6, C7, C9: C, symbol Device:C
- removed C10, C? (x2): 100 nF, symbol Device:C
- removed C?: 4.7 nF, symbol Device:C
- removed D1: 1v5_PWR, symbol Device:LED
- removed D2: 3v3_PWR, symbol Device:LED
- removed D3: 5v_PWR, symbol Device:LED
- removed FL?: Filter_EMI_LL_1423, symbol Device:Filter_EMI_LL_1423
- removed J1: USB_C_Receptacle_USB2.0, symbol Connector:USB_C_Receptacle_USB2.0
- removed J2: USB_GPIO, symbol Connector_Generic:Conn_01x06
- removed J?: Conn_01x02, symbol Connector_Generic:Conn_01x02
- removed JP1: I_3v3, symbol Jumper:Jumper_2_Bridged
- removed JP2: I_1v5, symbol Jumper:Jumper_2_Bridged
- removed JP3: USB_5v, symbol Jumper:Jumper_2_Bridged
- removed JP4: EEPROM_WR, symbol Jumper:Jumper_2_Bridged
- removed JP5: USB_TX, symbol Jumper:Jumper_2_Bridged
- removed JP6: USB_RX, symbol Jumper:Jumper_2_Bridged
- removed R1, R3: 5.1k, symbol Device:R
- removed R2, R4, R5, R? (x3): R, symbol Device:R
- removed R6, R7, R8: 10k, symbol Device:R
- removed R? (x3): 1k, symbol Device:R
- removed TP?: PHYCLK, symbol Connector:TestPoint
- removed U1: LM2940, Package_TO_SOT_THT:TO-220-3_Vertical, symbol old:LM2937xT
- removed U2: TL760, Package_TO_SOT_THT:TO-220-3_Vertical, symbol old:LM2937xT
- removed U3: LF15_TO252, Package_TO_SOT_SMD:TO-252-2, symbol Regulator_Linear:LF15_TO252
- removed U4: M24C02-WMN, Package_SO:SOIC-8_3.9x4.9mm_P1.27mm, symbol Memory_EEPROM:M24C02-WMN
- removed U5: XR21V1410, symbol viaems-parts:XR21V1410
- removed U6: TJA1101B, Package_DFN_QFN:QFN-36-1EP_6x6mm_P0.5mm_EP3.7x3.7mm, symbol viaems-parts:TJA1101B
- added C24, C25, C26, C27, C28, C29, C30, C31, C32, C33, C34, C35, C36, C37, C38: C, Capacitor_SMD:C_0805_2012Metric, symbol Device:C
- added J10, J11, J4, J5, J6, J7, J8, J9: Conn_02x08_Counter_Clockwise, Connector_PinHeader_2.54mm:PinHeader_2x08_P2.54mm_Vertical, symbol Connector_Generic:Conn_02x08_Odd_Even
- added JP7: VDD_HV_A_SEL, Connector_PinHeader_2.54mm:PinHeader_1x03_P2.54mm_Vertical, symbol Jumper:Jumper_3_Bridged12
- added R23: R, Resistor_SMD:R_0805_2012Metric, symbol Device:R
- added TP2: TP_1V1, TestPoint:TestPoint_Pad_D1.5mm, symbol Connector:TestPoint
- added TP3: TP_2V5, TestPoint:TestPoint_Pad_D1.5mm, symbol Connector:TestPoint
- added U7: S32K344, viaems-parts:IC_S32K344NHT1MPBST, symbol viaems-boards:S32K344
- added Y1: 8 MHz, Crystal:Crystal_HC49-U_Vertical, symbol Device:Crystal
- C2, C8: footprint (none) -> Capacitor_SMD:C_0805_2012Metric
Connections:
- net 3v3: now also C35.1, C36.1, C37.1, JP7.3 (B), U7.38 (VDD_HV_B), U7.57 (VDD_HV_B), U7.77 (VDD_HV_B)
- net 5v: now also JP7.1 (A); no longer C8.1
- net GND: now also C24.2, C25.2, C26.2, C27.2, C28.2, C29.2, C30.2, C31.2, C38.2, U7.107 (VSS), U7.127 (VSS), U7.150 (VSS), U7.168 (VSS), U7.17 (VREFL), U7.22 (VSS), U7.24 (VSS), U7.37 (VSS), U7.58 (VSS), U7.78 (VSS)
- net Vin: no longer names the net of C2.1
- net Vin: now also R23.1, Y1.1
- new net: C32.2, C33.2, C34.2
- new net: C8.1, U7.23 (EXTAL), Y1.2
- new net: C24.1, C25.1, C26.1, C27.1, TP2.1, U7.106 (V11), U7.149 (V11), U7.21 (V11), U7.59 (V11)
- new net: C35.2, C36.2, C37.2
- new net: R23.2, U7.25 (XTAL)
- new net: C31.1, TP3.1, U7.19 (V25)
- new net PTA0: J9.16 (Pin_16), U7.137 (PTA0)
- new net PTA1: J9.12 (Pin_12), U7.135 (PTA1)
- new net PTA10: U7.161 (PTA10)
- new net PTA11: J8.11 (Pin_11), U7.160 (PTA11)
- new net PTA12: J8.13 (Pin_13), U7.159 (PTA12)
- new net PTA13: J8.12 (Pin_12), U7.155 (PTA13)
- new net PTA14: J8.6 (Pin_6), U7.152 (PTA14)
- new net PTA15: J9.1 (Pin_1), U7.145 (PTA15)
- new net PTA16: J9.5 (Pin_5), U7.143 (PTA16)
- new net PTA17: J11.5 (Pin_5), U7.109 (PTA17)
- new net PTA18: J5.1 (Pin_1), U7.1 (PTA18)
- new net PTA19: J5.2 (Pin_2), U7.2 (PTA19)
- new net PTA2: J10.7 (Pin_7), U7.124 (PTA2)
- new net PTA20: J5.4 (Pin_4), U7.3 (PTA20)
- new net PTA21: J5.5 (Pin_5), U7.6 (PTA21)
- new net PTA24: J5.13 (Pin_13), U7.14 (PTA24)
- new net PTA25: J5.16 (Pin_16), U7.15 (PTA25)
- new net PTA27: J4.3 (Pin_3), U7.28 (PTA27)
- new net PTA28: J4.5 (Pin_5), U7.30 (PTA28)
- new net PTA29: J4.7 (Pin_7), U7.32 (PTA29)
- new net PTA3: J10.9 (Pin_9), U7.123 (PTA3)
- new net PTA30: J4.8 (Pin_8), U7.33 (PTA30)
- new net PTA31: J4.10 (Pin_10), U7.39 (PTA31)
- new net PTA4: U7.170 (PTA4)
- new net PTA5: U7.167 (PTA5)
- new net PTA6: J11.11 (Pin_11), U7.102 (PTA6)
- new net PTA7: J11.15 (Pin_15), U7.100 (PTA7)
- new net PTA8: J8.1 (Pin_1), U7.172 (PTA8)
- new net PTA9: J8.3 (Pin_3), U7.171 (PTA9)
- new net PTB0: J11.8 (Pin_8), U7.95 (PTB0)
- new net PTB1: J11.6 (Pin_6), U7.94 (PTB1)
- new net PTB10: J10.1 (Pin_1), U7.129 (PTB10)
- new net PTB11: J10.3 (Pin_3), U7.126 (PTB11)
- new net PTB12: J10.12 (Pin_12), U7.117 (PTB12)
- new net PTB13: J10.10 (Pin_10), U7.116 (PTB13)
- new net PTB14: J10.6 (Pin_6), U7.114 (PTB14)
- new net PTB15: J10.4 (Pin_4), U7.113 (PTB15)
- new net PTB16: J10.2 (Pin_2), U7.112 (PTB16)
- new net PTB17: J11.3 (Pin_3), U7.110 (PTB17)
- new net PTB18: J4.13 (Pin_13), U7.42 (PTB18)
- new net PTB19: J4.14 (Pin_14), U7.43 (PTB19)
- new net PTB2: U7.79 (PTB2)
- new net PTB20: U7.44 (PTB20)
- new net PTB21: U7.45 (PTB21)
- new net PTB22: U7.67 (PTB22)
- new net PTB23: U7.69 (PTB23)
- new net PTB24: U7.70 (PTB24)
- new net PTB25: U7.72 (PTB25)
- new net PTB26: U7.73 (PTB26)
- new net PTB27: U7.75 (PTB27)
- new net PTB28: U7.76 (PTB28)
- new net PTB29: U7.80 (PTB29)
- new net PTB3: U7.74 (PTB3)
- new net PTB4: U7.48 (PTB4)
- new net PTB5: U7.47 (PTB5)
- new net PTB8: J9.8 (Pin_8), U7.133 (PTB8)
- new net PTB9: J9.2 (Pin_2), U7.130 (PTB9)
- new net PTC0: U7.62 (PTC0)
- new net PTC1: U7.61 (PTC1)
- new net PTC10: J11.2 (Pin_2), U7.92 (PTC10)
- new net PTC11: U7.90 (PTC11)
- new net PTC12: U7.83 (PTC12)
- new net PTC13: U7.81 (PTC13)
- new net PTC14: U7.71 (PTC14)
- new net PTC15: U7.68 (PTC15)
- new net PTC16: U7.66 (PTC16)
- new net PTC17: U7.65 (PTC17)
- new net PTC18: U7.82 (PTC18)
- new net PTC19: U7.84 (PTC19)
- new net PTC2: U7.50 (PTC2)
- new net PTC20: U7.85 (PTC20)
- new net PTC21: U7.86 (PTC21)
- new net PTC23: U7.87 (PTC23)
- new net PTC24: U7.88 (PTC24)
- new net PTC25: U7.89 (PTC25)
- new net PTC26: U7.91 (PTC26)
- new net PTC27: J11.4 (Pin_4), U7.93 (PTC27)
- new net PTC28: J11.10 (Pin_10), U7.96 (PTC28)
- new net PTC29: J11.16 (Pin_16), U7.99 (PTC29)
- new net PTC3: U7.49 (PTC3)
- new net PTC30: J11.13 (Pin_13), U7.101 (PTC30)
- new net PTC31: J11.9 (Pin_9), U7.103 (PTC31)
- new net PTC4: U7.166 (PTC4)
- new net PTC5: U7.165 (PTC5)
- new net PTC6: J9.9 (Pin_9), U7.141 (PTC6)
- new net PTC7: J9.11 (Pin_11), U7.140 (PTC7)
- new net PTC8: J11.14 (Pin_14), U7.98 (PTC8)
- new net PTC9: J11.12 (Pin_12), U7.97 (PTC9)
- new net PTD0: J5.7 (Pin_7), U7.8 (PTD0)
- new net PTD1: J5.8 (Pin_8), U7.7 (PTD1)
- new net PTD10: U7.56 (PTD10)
- new net PTD11: U7.55 (PTD11)
- new net PTD12: U7.54 (PTD12)
- new net PTD13: J4.12 (Pin_12), U7.41 (PTD13)
- new net PTD14: J4.11 (Pin_11), U7.40 (PTD14)
- new net PTD15: J4.9 (Pin_9), U7.35 (PTD15)
- new net PTD16: U7.34 (PTD16)
- new net PTD17: J4.6 (Pin_6), U7.31 (PTD17)
- new net PTD2: J10.13 (Pin_13), U7.121 (PTD2)
- new net PTD20: J11.1 (Pin_1), U7.111 (PTD20)
- new net PTD21: J10.8 (Pin_8), U7.115 (PTD21)
- new net PTD22: J10.14 (Pin_14), U7.118 (PTD22)
- new net PTD23: J10.11 (Pin_11), U7.122 (PTD23)
- new net PTD24: J10.5 (Pin_5), U7.125 (PTD24)
- new net PTD26: J9.4 (Pin_4), U7.131 (PTD26)
- new net PTD27: J9.6 (Pin_6), U7.132 (PTD27)
- new net PTD28: J9.10 (Pin_10), U7.134 (PTD28)
- new net PTD29: J9.14 (Pin_14), U7.136 (PTD29)
- new net PTD3: J10.15 (Pin_15), U7.120 (PTD3)
- new net PTD30: J9.15 (Pin_15), U7.138 (PTD30)
- new net PTD31: J9.13 (Pin_13), U7.139 (PTD31)
- new net PTD4: J10.16 (Pin_16), U7.119 (PTD4)
- new net PTD5: U7.53 (PTD5)
- new net PTD6: U7.52 (PTD6)
- new net PTD7: U7.51 (PTD7)
- new net PTD8: U7.64 (PTD8)
- new net PTD9: U7.63 (PTD9)
- new net PTE0: J8.7 (Pin_7), U7.163 (PTE0)
- new net PTE1: J8.9 (Pin_9), U7.162 (PTE1)
- new net PTE10: J5.9 (Pin_9), U7.10 (PTE10)
- new net PTE11: J5.10 (Pin_10), U7.9 (PTE11)
- new net PTE12: J4.4 (Pin_4), U7.29 (PTE12)
- new net PTE13: J5.12 (Pin_12), U7.11 (PTE13)
- new net PTE14: J4.1 (Pin_1), U7.26 (PTE14)
- new net PTE15: J5.6 (Pin_6), U7.5 (PTE15)
- new net PTE16: J5.3 (Pin_3), U7.4 (PTE16)
- new net PTE17: J9.7 (Pin_7), U7.142 (PTE17)
- new net PTE18: J9.3 (Pin_3), U7.144 (PTE18)
- new net PTE2: J8.4 (Pin_4), U7.147 (PTE2)
- new net PTE21: J8.8 (Pin_8), U7.153 (PTE21)
- new net PTE22: J8.10 (Pin_10), U7.154 (PTE22)
- new net PTE23: J8.14 (Pin_14), U7.156 (PTE23)
- new net PTE24: J8.16 (Pin_16), U7.157 (PTE24)
- new net PTE25: J8.15 (Pin_15), U7.158 (PTE25)
- new net PTE26: J8.5 (Pin_5), U7.164 (PTE26)
- new net PTE3: J4.2 (Pin_2), U7.27 (PTE3)
- new net PTE4: J5.14 (Pin_14), U7.13 (PTE4)
- new net PTE5: J5.11 (Pin_11), U7.12 (PTE5)
- new net PTE6: J8.2 (Pin_2), U7.146 (PTE6)
- new net PTE7: J11.7 (Pin_7), U7.104 (PTE7)
- new net PTE8: U7.46 (PTE8)
- new net PTE9: U7.36 (PTE9)
- new net Power/1v5: C28.1, C29.1, C30.1, U7.105 (V15), U7.148 (V15), U7.20 (V15), U7.60 (V15)
- new net VDD_HV_A: C32.1, C33.1, C34.1, C38.1, JP7.2 (C), U7.108 (VDD_HV_AP), U7.128 (VDD_HV_A), U7.151 (VDD_HV_A), U7.16 (VREFH), U7.169 (VDD_HV_A), U7.18 (VDD_HV_A)
- no-connect marks 8 -> 0
Other:
- removed sheet CPU
- added sheet Debug (debug.kicad_sch)
- added sheet Ethernet (ethernet.kicad_sch)
- added sheet Power (power.kicad_sch)
- added sheet USB (usb.kicad_sch)
- note added: "Default configuration uses 5v for VDD_HV_A and 3.3v for VDD_HV_B. Optionally, 3.3v can be used for HDD_HV_A if JP7 is set to 2-3."
- note removed: "MII_MODE - 10 - RMII Mode, 50 MHz REF_CLK Out"

Commit message: more
Connections:
- net PTB2: now also J6.13 (Pin_13)
- net PTB20: now also J4.16 (Pin_16)
- net PTB21: now also J4.15 (Pin_15)
- net PTB22: now also J7.7 (Pin_7)
- net PTB23: now also J7.5 (Pin_5)
- net PTB24: now also J7.4 (Pin_4)
- net PTB25: now also J7.2 (Pin_2)
- net PTB26: now also J7.1 (Pin_1)
- net PTB27: now also J6.15 (Pin_15)
- net PTB28: now also J6.14 (Pin_14)
- net PTB29: now also J6.12 (Pin_12)
- net PTB3: now also J6.16 (Pin_16)
- net PTC11: now also J6.2 (Pin_2)
- net PTC12: now also J6.9 (Pin_9)
- net PTC13: now also J6.11 (Pin_11)
- net PTC14: now also J7.3 (Pin_3)
- net PTC18: now also J6.10 (Pin_10)
- net PTC19: now also J6.8 (Pin_8)
- net PTC20: now also J6.7 (Pin_7)
- net PTC21: now also J6.6 (Pin_6)
- net PTC23: now also J6.5 (Pin_5)
- net PTC24: now also J6.4 (Pin_4)
- net PTC25: now also J6.3 (Pin_3)
- net PTC26: now also J6.1 (Pin_1)

Commit message: more
Parts:
- U7: symbol viaems-boards:S32K344 -> viaems-parts:S32K344
Connections:
- net PTB22: now also J7.6 (Pin_6); no longer J7.7 (Pin_7)
- net PTC3: now also J7.10 (Pin_10)
- net PTD5: now also J7.9 (Pin_9)
- net PTD8: now also J7.7 (Pin_7)
- net PTD9: now also J7.8 (Pin_8)
- no-connect marks 0 -> 7
