File: proto-s323k44/debug.kicad_sch (KiCad schematic)
At the start: 11 parts, among them J13 TRACE

Commit message: more
Connections:
- net GND: now also J13.11 (GND), J13.13 (GND), J13.15 (GND), J13.17 (GND), J13.19 (GND), J13.5 (GND)
Changed lines of the file:
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@@
+	)
+	(junction
+		(at 76.2 119.38)
+		(diameter 0)
+		(color 0 0 0 0)
+	)
+	(junction
+		(at 71.12 119.38)
+		(diameter 0)
+		(color 0 0 0 0)
 	)
 	(junction
@@
 	)
 	(junction
+		(at 78.74 119.38)
+		(diameter 0)
+		(color 0 0 0 0)
+	)
+	(junction
+		(at 73.66 119.38)
+		(diameter 0)
+		(color 0 0 0 0)
+	)
+	(junction
+		(at 81.28 119.38)
+		(diameter 0)
+		(color 0 0 0 0)
+	)
+	(junction
 		(at 115.57 90.17)
 		(diameter 0)
@@
 	(wire
 		(pts
+			(xy 76.2 119.38) (xy 73.66 119.38)
+		)
+		(stroke
+			(width 0)
+			(type default)
+		)
+	)
+	(wire
+		(pts
+			(xy 76.2 119.38) (xy 76.2 118.11)
+		)
+		(stroke
+			(width 0)
+			(type default)
+		)
+	)
+	(wire
+		(pts
 			(xy 111.76 97.79) (xy 130.81 97.79)
 		)
@@
 	(wire
 		(pts
+			(xy 71.12 119.38) (xy 66.04 119.38)
+		)
+		(stroke
+			(width 0)
+			(type default)
+		)
+	)
+	(wire
+		(pts
 			(xy 130.81 74.93) (xy 130.81 76.2)
 		)
@@
 	(wire
 		(pts
+			(xy 73.66 119.38) (xy 71.12 119.38)
+		)
+		(stroke
+			(width 0)
+			(type default)
+		)
+	)
+	(wire
+		(pts
+			(xy 83.82 118.11) (xy 83.82 119.38)
+		)
+		(stroke
+			(width 0)
+			(type default)
+		)
+	)
+	(wire
+		(pts
 			(xy 86.36 74.93) (xy 86.36 82.55)
 		)
@@
 	(wire
 		(pts
+			(xy 71.12 119.38) (xy 71.12 118.11)
+		)
+		(stroke
+			(width 0)
+			(type default)
+		)
+	)
+	(wire
+		(pts
 			(xy 138.43 83.82) (xy 138.43 100.33)
 		)
@@
 	(wire
 		(pts
+			(xy 81.28 119.38) (xy 78.74 119.38)
+		)
+		(stroke
+			(width 0)
+			(type default)
+		)
+	)
+	(wire
+		(pts
 			(xy 123.19 74.93) (xy 130.81 74.93)
 		)
@@
 	(wire
 		(pts
+			(xy 78.74 119.38) (xy 78.74 118.11)
+		)
+		(stroke
+			(width 0)
+			(type default)
+		)
+	)
+	(wire
+		(pts
+			(xy 78.74 119.38) (xy 76.2 119.38)
+		)
+		(stroke
+			(width 0)
+			(type default)
+		)
+	)
+	(wire
+		(pts
 			(xy 99.06 97.79) (xy 104.14 97.79)
 		)
@@
 	(wire
 		(pts
+			(xy 66.04 119.38) (xy 66.04 107.95)
+		)
+		(stroke
+			(width 0)
+			(type default)
+		)
+	)
+	(wire
+		(pts
 			(xy 99.06 100.33) (xy 104.14 100.33)
 		)
@@
 		)
 		(stroke
+			(width 0)
+			(type default)
+		)
+	)
+	(wire
+		(pts
+			(xy 73.66 119.38) (xy 73.66 118.11)
+		)
+		(stroke

Commit message: more
Parts:
- removed R29, R30, R31, R32, R37: 22, Resistor_SMD:R_0805_2012Metric, symbol Device:R
- J13: symbol viaems-boards:Conn_ARM_ETM_SWD_20 -> viaems-parts:Conn_ARM_ETM_SWD_20
Connections:
- net TCK: now also J13.4 (SWDCLK/TCK), R38.1
- net TDI: now also J13.8 (TDI); no longer R38.1
- net TDO: now also J13.6 (SWO/TDO)
- net TMS: now also J13.2 (SWDIO/TMS)
- net nRESET: now also J13.10 (~{RESET})
Other:
- moved on the sheet: R34, R35, R36, R38, R8
