File: proto-s323k44/ethernet.kicad_sch (KiCad schematic)
At the start: 32 parts, among them J12 RMII, J3 ETH, U6 TJA1101B, U8 KC2520Z

Commit message: more
Connections:
- no-connect marks 7 -> 8
Changed lines of the file:
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@@
 	)
 	(junction
+		(at 129.54 45.72)
+		(diameter 0)
+		(color 0 0 0 0)
+	)
+	(junction
 		(at 78.74 31.75)
 		(diameter 0)
@@
 	)
 	(no_connect
+		(at 96.52 57.15)
+	)
+	(no_connect
 		(at 96.52 67.31)
 	)
@@
 	(wire
 		(pts
-			(xy 111.76 45.72) (xy 138.43 45.72)
+			(xy 111.76 45.72) (xy 129.54 45.72)
 		)
 		(stroke
@@
 	(wire
 		(pts
+			(xy 129.54 45.72) (xy 138.43 45.72)
+		)
+		(stroke
+			(width 0)
+			(type default)
+		)
+	)
+	(wire
+		(pts
 			(xy 111.76 113.03) (xy 111.76 111.76)
 		)
@@
 					(unit 1)
 				)
+			)
+		)
+	)
+	(symbol
+		(lib_id "power:PWR_FLAG")
+		(at 129.54 45.72 180)
+		(unit 1)
+		(exclude_from_sim no)
+		(in_bom yes)
+		(on_board yes)
+		(dnp no)
+		(fields_autoplaced yes)
+		(property "Reference" "#FLG05"
+			(at 129.54 47.625 0)
+			(effects
+				(font
+					(size 1.27 1.27)
+				)
+				(hide yes)
+			)
+		)
+		(property "Value" "PWR_FLAG"
+			(at 129.54 50.8 0)
+			(effects
+				(font
+					(size 1.27 1.27)
+				)
+				(hide yes)
+			)
+		)
+		(property "Footprint" ""
+			(at 129.54 45.72 0)
+			(effects
+				(font
+					(size 1.27 1.27)
+				)
+				(hide yes)
+			)
+		)
+		(property "Datasheet" "~"
+			(at 129.54 45.72 0)
+			(effects
+				(font
+					(size 1.27 1.27)
+				)
+				(hide yes)
+			)
+		)
+		(property "Description" "Special symbol for telling ERC where power comes from"
+			(at 129.54 45.72 0)
+			(effects
+				(font
+					(size 1.27 1.27)
+				)
+				(hide yes)
+			)
+		)
+		(pin "1"
+		)
+		(instances
+			(project ""
+				(path "/11f330e8-2377-4dd2-90f0-6a90097d4fa1/9ca8e9fb-b557-42ab-9be2-8722d4d40f19"
+					(reference "#FLG05")
+					(unit 1)
+				)

Commit message: more
Connections:
- net GND: now also U6.6 (XI); no longer U6.5 (XO)
- net at TP1.1, U6.20 (CLK_IN_OUT): now also U8.3 (CLK)
- net at U6.12 (TRX_P): now also FL1.3; no longer FL1.4
- net at C11.1: now also FL1.4; no longer FL1.3
- no-connect marks 8 -> 9
Other:
- moved on the sheet: TP1
Changed lines of the file:
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@@
 	)
 	(junction
+		(at 154.94 100.33)
+		(diameter 0)
+		(color 0 0 0 0)
+	)
+	(junction
 		(at 87.63 31.75)
 		(diameter 0)
@@
 		(at 96.52 72.39)
 	)
+	(no_connect
+		(at 128.27 105.41)
+	)
 	(wire
 		(pts
@@
 	(wire
 		(pts
+			(xy 154.94 100.33) (xy 128.27 100.33)
+		)
+		(stroke
+			(width 0)
+			(type default)
+		)
+	)
+	(wire
+		(pts
 			(xy 33.02 69.85) (xy 59.69 69.85)
 		)
@@
 	(wire
 		(pts
-			(xy 128.27 102.87) (xy 170.18 102.87)
-		)
-		(stroke
-			(width 0)
-			(type default)
-		)
-	)
-	(wire
-		(pts
 			(xy 81.28 40.64) (xy 87.63 40.64)
 		)
@@
 	(wire
 		(pts
-			(xy 128.27 105.41) (xy 130.81 105.41)
+			(xy 128.27 102.87) (xy 130.81 102.87)
 		)
 		(stroke
@@
 	(wire
 		(pts
-			(xy 135.255 100.33) (xy 135.255 99.695)
-		)
-		(stroke
-			(width 0)
-			(type default)
-		)
-	)
-	(wire
-		(pts
 			(xy 139.065 69.215) (xy 143.51 69.215)
 		)
@@
 	(wire
 		(pts
+			(xy 170.18 100.33) (xy 170.18 116.84)
+		)
+		(stroke
+			(width 0)
+			(type default)
+		)
+	)
+	(wire
+		(pts
 			(xy 46.99 54.61) (xy 46.99 82.55)
 		)
@@
 	(wire
 		(pts
-			(xy 170.18 102.87) (xy 170.18 116.84)
-		)
-		(stroke
-			(width 0)
-			(type default)
-		)
-	)
-	(wire
-		(pts
 			(xy 46.99 44.45) (xy 40.64 44.45)
 		)
@@
 	(wire
 		(pts
+			(xy 170.18 100.33) (xy 154.94 100.33)
+		)
+		(stroke
+			(width 0)
+			(type default)
+		)
+	)
+	(wire
+		(pts
 			(xy 44.45 85.09) (xy 96.52 85.09)
 		)
@@
 	(wire
 		(pts
-			(xy 128.27 100.33) (xy 135.255 100.33)
-		)
-		(stroke
-			(width 0)
-			(type default)
-		)
-	)
-	(wire
-		(pts
 			(xy 129.54 45.72) (xy 138.43 45.72)
 		)
@@
 			)
 		)
-		(property "Description" ""
+		(property "Description" "Unpolarized capacitor"
 			(at 161.925 74.295 0)
 			(effects
@@
 			)
 		)
-		(property "Description" ""
+		(property "Description" "Resistor"
 			(at 173.355 94.615 0)
 			(effects
@@
 			)
 		)
-		(property "Description" ""
+		(property "Description" "Power symbol creates a global label with name \"GND\" , ground"
 			(at 173.355 98.425 0)
 			(effects
@@
 			)
 		)
-		(property "Description" ""
+		(property "Description" "Generic connector, single row, 01x02, script generated (kicad-library-utils/schlib/autogen/connector/)"
 			(at 198.755 71.12 0)
 			(effects
@@
 	(symbol
 		(lib_id "Connector:TestPoint")
-		(at 135.255 99.695 0)
+		(at 154.94 100.33 0)
 		(unit 1)
 		(exclude_from_sim no)
@@
 		(dnp no)
 		(property "Reference" "TP1"
-			(at 136.652 95.5583 0)
+			(at 156.337 96.1933 0)
 			(effects
 				(font
@@
 		)
 		(property "Value" "PHYCLK"
-			(at 136.652 98.0952 0)
+			(at 156.337 98.7302 0)
 			(effects
 				(font
@@
 		)
 		(property "Footprint" "TestPoint:TestPoint_Pad_D1.5mm"
-			(at 140.335 99.695 0)
+			(at 160.02 100.33 0)
 			(effects
 				(font
@@
 		)
 		(property "Datasheet" "~"
-			(at 140.335 99.695 0)
+			(at 160.02 100.33 0)
 			(effects
 				(font
@@
 			)
 		)
-		(property "Description" ""
-			(at 135.255 99.695 0)
+		(property "Description" "test point"
+			(at 154.94 100.33 0)
 			(effects
 				(font
@@
 			)
 		)
-		(property "Description" ""
+		(property "Description" "Unpolarized capacitor"
 			(at 181.61 94.615 0)
 			(effects
@@
 			)
 		)
-		(property "Description" ""
+		(property "Description" "Power symbol creates a global label with name \"GND\" , ground"
 			(at 110.49 116.84 0)
 			(effects
@@
 			)
 		)
-		(property "Description" ""
+		(property "Description" "Power symbol creates a global label with name \"GND\" , ground"
 			(at 81.28 41.91 0)
 			(effects
@@
 	(symbol
 		(lib_id "power:GND")
-		(at 130.81 105.41 0)
+		(at 130.81 102.87 0)
 		(unit 1)
 		(exclude_from_sim no)
@@
 		(fields_autoplaced yes)
 		(property "Reference" "#PWR08"
-			(at 130.81 111.76 0)
+			(at 130.81 109.22 0)
 			(effects
 				(font
@@
 		)
 		(property "Value" "GND"
-			(at 130.81 110.49 0)
+			(at 130.81 107.95 0)
 			(effects
 				(font
@@
 		)
 		(property "Footprint" ""
-			(at 130.81 105.41 0)
+			(at 130.81 102.87 0)
 			(effects
 				(font
@@
 		)
 		(property "Datasheet" ""
-			(at 130.81 105.41 0)
+			(at 130.81 102.87 0)
 			(effects
 				(font
@@
 		)
 		(property "Description" "Power symbol creates a global label with name \"GND\" , ground"
-			(at 130.81 105.41 0)
+			(at 130.81 102.87 0)
 			(effects
 				(font
@@
 			)
 		)
-		(property "Description" ""
+		(property "Description" "Power symbol creates a global label with name \"GND\" , ground"
 			(at 83.82 95.25 0)
 			(effects
@@
 			)
 		)
-		(property "Description" ""
+		(property "Description" "Power symbol creates a global label with name \"GND\" , ground"
 			(at 26.67 171.45 0)
 			(effects
@@
 			)
 		)
-		(property "Description" ""
+		(property "Description" "Resistor"
 			(at 89.535 93.98 0)
 			(effects
@@
 			)
 		)
-		(property "Description" ""
+		(property "Description" "Resistor"
 			(at 181.61 82.55 0)
 			(effects
@@
 			)
 		)
-		(property "Description" ""
+		(property "Description" "Unpolarized capacitor"
 			(at 161.925 69.215 0)
 			(effects
@@
 			)
 		)
-		(property "Description" ""
+		(property "Description" "Power symbol creates a global label with name \"GND\" , ground"
 			(at 138.43 53.34 0)
 			(effects
@@
 			)
 		)
-		(property "Description" ""
+		(property "Description" "Power symbol creates a global label with name \"GND\" , ground"
 			(at 34.29 107.95 0)
 			(effects
@@
 			)
 		)
-		(property "Description" ""
+		(property "Description" "Resistor"
 			(at 173.355 82.55 0)
 			(effects
@@
 			)
 		)
-		(property "Description" ""
+		(property "Description" "Power symbol creates a global label with name \"GND\" , ground"
 			(at 69.85 171.45 0)
 			(effects
@@
 			)
 		)
-		(property "Description" ""
+		(property "Description" "Power symbol creates a global label with name \"GND\" , ground"
 			(at 181.61 98.425 0)
 			(effects
