File: proto-s323k44/proto-s32k344.kicad_pcb (KiCad board)
At the start: 2 copper layers, 46.4 x 99.6 mm, 104 parts, among them J1 USB_C_Receptacle_USB2.0, J10 Conn_02x08_Counter_Clockwise, J11 Conn_02x08_Counter_Clockwise, J12 RMII, J13 TRACE, J15 5v_in, J2 USB_GPIO, J3 ETH, J4 Conn_02x08_Counter_Clockwise, J5 Conn_02x08_Counter_Clockwise, J6 Conn_02x08_Counter_Clockwise, J7 Conn_02x08_Counter_Clockwise, J8 Conn_02x08_Counter_Clockwise, J9 Conn_02x08_Counter_Clockwise, U2 TL760, U3 LF15_TO252, U4 M24C02-WMN, U5 XR21V1410, U6 TJA1101B, U7 S32K344, U8 KC2520Z, Y1 8 MHz

Commit message: more
Connections:
- J12 pad 7: /PTC15 -> /PTC17
- J4 pad 15: unconnected-(J4-Pin_15-Pad15) -> /PTB21
- J4 pad 16: unconnected-(J4-Pin_16-Pad16) -> /PTB20
- J6 pad 1: unconnected-(J6-Pin_1-Pad1) -> /PTC26
- J6 pad 10: unconnected-(J6-Pin_10-Pad10) -> /PTC18
- J6 pad 11: unconnected-(J6-Pin_11-Pad11) -> /PTC13
- J6 pad 12: unconnected-(J6-Pin_12-Pad12) -> /PTB29
- J6 pad 13: unconnected-(J6-Pin_13-Pad13) -> /PTB2
- J6 pad 14: unconnected-(J6-Pin_14-Pad14) -> /PTB28
- J6 pad 15: unconnected-(J6-Pin_15-Pad15) -> /PTB27
- J6 pad 16: unconnected-(J6-Pin_16-Pad16) -> /PTB3
- J6 pad 2: unconnected-(J6-Pin_2-Pad2) -> /PTC11
- J6 pad 3: unconnected-(J6-Pin_3-Pad3) -> /PTC25
- J6 pad 4: unconnected-(J6-Pin_4-Pad4) -> /PTC24
- J6 pad 5: unconnected-(J6-Pin_5-Pad5) -> /PTC23
- J6 pad 6: unconnected-(J6-Pin_6-Pad6) -> /PTC21
- J6 pad 7: unconnected-(J6-Pin_7-Pad7) -> /PTC20
- J6 pad 8: unconnected-(J6-Pin_8-Pad8) -> /PTC19
- J6 pad 9: unconnected-(J6-Pin_9-Pad9) -> /PTC12
- J7 pad 1: unconnected-(J7-Pin_1-Pad1) -> /PTB26
- J7 pad 2: unconnected-(J7-Pin_2-Pad2) -> /PTB25
- J7 pad 3: unconnected-(J7-Pin_3-Pad3) -> /PTC14
- J7 pad 4: unconnected-(J7-Pin_4-Pad4) -> /PTB24
- J7 pad 5: unconnected-(J7-Pin_5-Pad5) -> /PTB23
- J7 pad 7: unconnected-(J7-Pin_7-Pad7) -> /PTB22
- JP5 pad 2: /USB/UART_TX -> /PTC15
- JP6 pad 2: /USB/UART_RX -> /PTC16
- R17 pad 1: /PTC15 -> /PTC17
- U6 pad 18: /PTC15 -> /PTC17
Routing:
- net /PTC17: track 0.00 -> 57.1 mm
- net /PTC16: track 0.00 -> 38.7 mm
- net /PTB21: track 0.00 -> 32.7 mm, vias 0 -> 2
- net /PTB20: track 0.00 -> 31.1 mm, vias 0 -> 2
- net /PTB22: track 0.00 -> 23.2 mm, vias 0 -> 2
- net /PTB24: track 0.00 -> 21.2 mm
- net /PTB23: track 0.00 -> 20.5 mm
- net /PTC15: track 57.4 -> 37.5 mm
- net /PTB25: track 0.00 -> 19.1 mm
- net /PTC14: track 0.00 -> 18.3 mm
- net /PTB26: track 0.00 -> 16.0 mm
- net /PTB3: track 0.00 -> 15.7 mm
- net /PTB28: track 0.00 -> 13.1 mm
- net /PTB27: track 0.00 -> 12.6 mm
- net /PTB29: track 0.00 -> 11.5 mm
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
Commit message: more
Parts:
- R33: moved to B.Cu
- moved JP1 111.9 mm to (90.6, 129.8), turned to 180 degrees
- moved JP2 106.8 mm to (90.5, 111.7)
- moved R33 55.3 mm to (76.1, 124.0), turned to -90 degrees
- moved JP6 32.0 mm to (96.3, 101.3)
- moved R20 20.9 mm to (37.6, 141.2)
- moved R4 7.32 mm to (89.7, 124.0)
- moved JP7 7.30 mm to (80.0, 109.7)
- moved R5 4.50 mm to (78.3, 126.0), turned to 90 degrees
- moved D2 4.06 mm to (91.8, 124.2)
- moved R2 3.30 mm to (89.8, 118.5)
- moved JP3 2.59 mm to (76.8, 132.1), turned to 180 degrees
- moved U2 2.52 mm to (84.7, 127.3)
- moved D3 2.00 mm to (80.3, 126.1), turned to -90 degrees
- moved U3 1.91 mm to (84.8, 116.9)
- moved D1 1.19 mm to (91.6, 118.5)
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Connections:
- J13 pad 11: unconnected-(J13-GND-Pad11) -> GND
- J13 pad 13: unconnected-(J13-GND-Pad13) -> GND
- J13 pad 15: unconnected-(J13-GND-Pad15) -> GND
- J13 pad 17: unconnected-(J13-GND-Pad17) -> GND
- J13 pad 19: unconnected-(J13-GND-Pad19) -> GND
- J13 pad 5: unconnected-(J13-GND-Pad5) -> GND
- J7 pad 10: unconnected-(J7-Pin_10-Pad10) -> /PTC3
- J7 pad 6: unconnected-(J7-Pin_6-Pad6) -> /PTB22
- J7 pad 7: /PTB22 -> /PTD8
- J7 pad 8: unconnected-(J7-Pin_8-Pad8) -> /PTD9
- J7 pad 9: unconnected-(J7-Pin_9-Pad9) -> /PTD5
Routing:
- net /3v3: track 0.00 -> 120.5 mm, vias 0 -> 5
- net /PTC16: track 38.7 -> 0.00 mm
- net /PTC15: track 37.5 -> 0.00 mm
- net /5v: track 0.00 -> 32.3 mm
- net /PTC3: track 0.00 -> 30.3 mm, vias 0 -> 2
- net /PTD9: track 0.00 -> 28.2 mm, vias 0 -> 2
- net /PTD5: track 0.00 -> 25.4 mm, vias 0 -> 2
- net /PTD8: track 0.00 -> 22.2 mm, vias 0 -> 2
- net /Power/1v5: track 0.00 -> 16.8 mm
- net /5v_usb: track 0.00 -> 15.0 mm
- net Net-(JP2-A): track 0.00 -> 9.19 mm
- net Net-(JP1-A): track 0.00 -> 4.65 mm
- net Net-(D2-A): track 0.00 -> 2.85 mm
- net Net-(U5-LOWPOWER): track 0.00 -> 2.69 mm, vias 0 -> 1
- net Net-(D1-A): track 0.00 -> 2.64 mm
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
Commit message: more
Parts:
- removed R29, R30, R31, R32, R37: 22, Resistor_SMD:R_0805_2012Metric
- U2: footprint Package_TO_SOT_SMD:TO-252-2 -> Package_TO_SOT_THT:TO-220-3_Vertical
- U4: footprint Package_SO:SO-8_3.9x4.9mm_P1.27mm -> Package_SO:SOIC-8_3.9x4.9mm_P1.27mm
- turned U7 to 0 degrees
Connections:
- FL1 pad 3: Net-(C11-Pad1) -> Net-(U6-TRX_P)
- FL1 pad 4: Net-(U6-TRX_P) -> Net-(C11-Pad1)
- J13 pad 10: Net-(J13-~{RESET}) -> /PTA5
- J13 pad 2: Net-(J13-SWDIO/TMS) -> /PTA4
- J13 pad 4: Net-(J13-SWDCLK/TCK) -> /PTC4
- J13 pad 6: Net-(J13-SWO/TDO) -> /PTA10
- J13 pad 8: Net-(J13-NC/TDI) -> /PTC5
- R38 pad 1: /PTC5 -> /PTC4
- U6 pad 5: GND -> unconnected-(U6-XO-Pad5)
- U6 pad 6: Net-(U6-XI) -> GND
- U8 pad 3: Net-(U6-XI) -> Net-(U6-CLK_IN_OUT)
Routing:
- net Net-(U6-XI): track 4.29 -> 0.00 mm
- net (no net): track 0.00 -> 4.29 mm
- net Net-(J13-SWDIO/TMS): track 3.32 -> 0.00 mm
- net /PTA4: track 11.1 -> 14.5 mm
- net Net-(J13-SWDCLK/TCK): track 3.05 -> 0.00 mm
- net /PTC4: track 8.56 -> 11.6 mm
- net Net-(J13-SWO/TDO): track 2.73 -> 0.00 mm
- net /PTA10: track 3.83 -> 6.56 mm
- net Net-(J13-~{RESET}): track 2.70 -> 0.00 mm
- net /PTA5: track 4.33 -> 7.03 mm
- net Net-(J13-NC/TDI): track 2.42 -> 0.00 mm
- net /PTC5: track 4.58 -> 7.01 mm
