File: proto-s323k44/usb.kicad_sch (KiCad schematic)
At the start: 13 parts, among them J1 USB_C_Receptacle_USB2.0, J2 USB_GPIO, U4 M24C02-WMN, U5 XR21V1410

Commit message: more
Parts:
- U4: footprint Package_SO:SO-8_3.9x4.9mm_P1.27mm -> Package_SO:SOIC-8_3.9x4.9mm_P1.27mm
Other:
- moved on the sheet: C9, R33, U5
