File: test-harness/test-harness.kicad_pcb (KiCad board)
At the start: 2 copper layers, 78 x 34 mm, 72 parts, among them J1 USB_C_Receptacle_USB2.0_16P, J2 Conn_ARM_JTAG_SWD_10, J3 Conn_01x16, J4 Conn_01x16, J5 Conn_01x06, J6 POWER, J7 POWER, U1 MachXO3D_9400, U2 FT2232H-56Q, U3 93CxxC, U4 TPS7B88Q1, Y1 12 MHz

Commit message: updates
Routing:
- net GND: track 95.3 -> 92.5 mm, vias 58 -> 61
