File: test-harness/test-harness.kicad_pcb (KiCad board)
At the start: 2 copper layers, 78 x 34 mm, 72 parts, among them J1 USB_C_Receptacle_USB2.0_16P, J2 Conn_ARM_JTAG_SWD_10, J3 Conn_01x16, J4 Conn_01x16, J5 Conn_01x06, J6 POWER, J7 POWER, U1 MachXO3D_9400, U2 FT2232H-56Q, U3 93CxxC, U4 TPS7B88Q1, Y1 12 MHz

Commit message: Test harness v2
Parts:
- removed ? (x4): , 
- added C35: C, Capacitor_SMD:C_0805_2012Metric, F.Cu at (82.3, 68.4)
- added C36: C, Capacitor_SMD:C_0805_2012Metric, F.Cu at (79.3, 68.4)
- added C37: C, Capacitor_SMD:C_0805_2012Metric, F.Cu at (112.4, 73.1)
- added C38: C, Capacitor_SMD:C_0805_2012Metric, F.Cu at (113.0, 68.2)
- added C39: C, Capacitor_SMD:C_0805_2012Metric, F.Cu at (110.8, 68.2)
- added C40: C, Capacitor_SMD:C_0805_2012Metric, F.Cu at (86.2, 116.9)
- added C41: C, Capacitor_SMD:C_0805_2012Metric, F.Cu at (113.2, 116.8)
- added C42: C, Capacitor_SMD:C_0805_2012Metric, F.Cu at (88.8, 121.1)
- added C43: C, Capacitor_SMD:C_0805_2012Metric, F.Cu at (115.8, 121.5)
- added C44: C, Capacitor_SMD:C_0805_2012Metric, F.Cu at (85.5, 121.2)
- added C45: C, Capacitor_SMD:C_0805_2012Metric, F.Cu at (112.7, 121.7)
- added C46: 0.1 uF, Capacitor_SMD:C_0805_2012Metric, F.Cu at (109.4, 91.4)
- added C47: 10 uF, Capacitor_SMD:C_0805_2012Metric, F.Cu at (109.4, 93.4)
- added C48: 0.1 uF, Capacitor_SMD:C_0805_2012Metric, F.Cu at (119.7, 92.0)
- added C49: 0.1 uF, Capacitor_SMD:C_0805_2012Metric, F.Cu at (118.6, 95.4)
- added D10: LED, LED_SMD:LED_0805_2012Metric, F.Cu at (81.0, 80.4)
- added D11: LED, LED_SMD:LED_0805_2012Metric, F.Cu at (83.5, 80.4)
- added D12: LED, LED_SMD:LED_0805_2012Metric, F.Cu at (103.6, 80.9)
- added D13: LED, LED_SMD:LED_0805_2012Metric, F.Cu at (106.4, 80.9)
- added D14: LED, LED_SMD:LED_0805_2012Metric, F.Cu at (108.9, 80.9)
- added D15: LED, LED_SMD:LED_0805_2012Metric, F.Cu at (111.4, 80.9)
- added D16: LED, LED_SMD:LED_0805_2012Metric, F.Cu at (113.9, 80.9)
- added D17: LED, LED_SMD:LED_0805_2012Metric, F.Cu at (116.6, 80.9)
- added D18: LED, LED_SMD:LED_0805_2012Metric, F.Cu at (119.1, 80.9)
- added D19: LED, LED_SMD:LED_0805_2012Metric, F.Cu at (121.7, 80.8)
- added D20: LED, LED_SMD:LED_0805_2012Metric, F.Cu at (119.1, 109.2)
- added D21: LED, LED_SMD:LED_0805_2012Metric, F.Cu at (93.2, 109.3)
- added D22: LED, LED_SMD:LED_0805_2012Metric, F.Cu at (116.5, 109.2)
- added D23: LED, LED_SMD:LED_0805_2012Metric, F.Cu at (90.7, 109.4)
- added D24: LED, LED_SMD:LED_0805_2012Metric, F.Cu at (113.9, 109.2)
- added D25: LED, LED_SMD:LED_0805_2012Metric, F.Cu at (88.1, 109.4)
- added D26: LED, LED_SMD:LED_0805_2012Metric, F.Cu at (111.2, 109.2)
- added D27: LED, LED_SMD:LED_0805_2012Metric, F.Cu at (85.6, 109.4)
- added D28: LED, LED_SMD:LED_0805_2012Metric, F.Cu at (108.6, 109.2)
- added D29: LED, LED_SMD:LED_0805_2012Metric, F.Cu at (83.0, 109.4)
- added D3: STATUS, LED_SMD:LED_0805_2012Metric, F.Cu at (69.6, 69.0)
- added D30: LED, LED_SMD:LED_0805_2012Metric, F.Cu at (106.0, 109.2)
- added D31: LED, LED_SMD:LED_0805_2012Metric, F.Cu at (80.5, 109.4)
- added D32: LED, LED_SMD:LED_0805_2012Metric, F.Cu at (103.4, 109.2)
- added D33: LED, LED_SMD:LED_0805_2012Metric, F.Cu at (77.9, 109.4)
- added D34: LED, LED_SMD:LED_0805_2012Metric, F.Cu at (101.1, 109.2)
- added D35: LED, LED_SMD:LED_0805_2012Metric, F.Cu at (75.4, 109.4)
- added D4: LED, LED_SMD:LED_0805_2012Metric, F.Cu at (93.6, 80.4)
- added D5: LED, LED_SMD:LED_0805_2012Metric, F.Cu at (91.1, 80.4)
- added D6: LED, LED_SMD:LED_0805_2012Metric, F.Cu at (86.0, 80.4)
- added D7: LED, LED_SMD:LED_0805_2012Metric, F.Cu at (88.6, 80.4)
- added D8: LED, LED_SMD:LED_0805_2012Metric, F.Cu at (75.9, 80.4)
- added D9: LED, LED_SMD:LED_0805_2012Metric, F.Cu at (78.4, 80.4)
- added H1: MountingHole, MountingHole:MountingHole_2.5mm_Pad, F.Cu at (58.8, 62.6)
- added H2: MountingHole, MountingHole:MountingHole_2.5mm_Pad, F.Cu at (127.8, 62.8)
- added H3: MountingHole, MountingHole:MountingHole_2.5mm_Pad, F.Cu at (58.8, 126.6)
- added H4: MountingHole, MountingHole:MountingHole_2.5mm_Pad, F.Cu at (127.8, 126.6)
- added J10: OUT_C, Connector_PinHeader_2.54mm:PinHeader_1x08_P2.54mm_Vertical, F.Cu at (120.2, 126.0)
- added J11: OUT_D, Connector_PinHeader_2.54mm:PinHeader_1x08_P2.54mm_Vertical, F.Cu at (93.7, 126.0)
- added J12: ANALOG1, Connector_PinHeader_2.54mm:PinHeader_1x04_P2.54mm_Vertical, F.Cu at (112.1, 87.8)
- added J13: ANALOG2, Connector_PinHeader_2.54mm:PinHeader_1x04_P2.54mm_Vertical, F.Cu at (119.8, 100.0)
- added J14: ANALOG3, Connector_PinHeader_2.54mm:PinHeader_1x04_P2.54mm_Vertical, F.Cu at (125.2, 83.0)
- added J15: ANALOG4, Connector_PinHeader_2.54mm:PinHeader_1x04_P2.54mm_Vertical, F.Cu at (125.2, 99.0)
- added J16: EXT, Connector_PinHeader_2.54mm:PinHeader_1x04_P2.54mm_Vertical, F.Cu at (100.0, 72.2)
- added J17: 5v_usb, Connector_PinHeader_2.54mm:PinHeader_1x02_P2.54mm_Vertical, F.Cu at (71.8, 123.8)
- added J8: 5v_usb, Connector_PinHeader_2.54mm:PinHeader_1x02_P2.54mm_Vertical, F.Cu at (67.8, 123.7)
- added J9: OUT_B, Connector_PinHeader_2.54mm:PinHeader_1x08_P2.54mm_Vertical, F.Cu at (105.2, 63.6)
- added JP1: DIR_A, Jumper:SolderJumper-3_P2.0mm_Open_TrianglePad1.0x1.5mm, F.Cu at (73.6, 69.0)
- added JP2: DIR_B, Jumper:SolderJumper-3_P2.0mm_Open_TrianglePad1.0x1.5mm, F.Cu at (102.0, 67.0)
- added JP3: DIR_C, Jumper:SolderJumper-3_P2.0mm_Open_TrianglePad1.0x1.5mm, F.Cu at (123.4, 119.6)
- added JP4: DIR_D, Jumper:SolderJumper-3_P2.0mm_Open_TrianglePad1.0x1.5mm, F.Cu at (95.8, 118.3)
- added JP5: ADC_EN, Jumper:SolderJumper-2_P1.3mm_Open_TrianglePad1.0x1.5mm, F.Cu at (103.4, 88.0)
- added R19: R, Resistor_SMD:R_0805_2012Metric, F.Cu at (69.6, 72.0)
- added R20: R, Resistor_SMD:R_0805_2012Metric, F.Cu at (78.3, 72.9)
- added R21: R, Resistor_SMD:R_0805_2012Metric, F.Cu at (76.6, 68.5)
- added R22: R, Resistor_SMD:R_0805_2012Metric, F.Cu at (93.6, 76.9)
- added R23: R, Resistor_SMD:R_0805_2012Metric, F.Cu at (91.1, 76.9)
- added R24: R, Resistor_SMD:R_0805_2012Metric, F.Cu at (86.0, 76.9)
- added R25: R, Resistor_SMD:R_0805_2012Metric, F.Cu at (88.6, 76.9)
- added R26: 3.3k, Resistor_SMD:R_0805_2012Metric, F.Cu at (75.9, 76.9)
- added R27: 3.3k, Resistor_SMD:R_0805_2012Metric, F.Cu at (78.4, 76.9)
- added R28: 3.3k, Resistor_SMD:R_0805_2012Metric, F.Cu at (81.0, 76.9)
- added R29: 3.3k, Resistor_SMD:R_0805_2012Metric, F.Cu at (83.5, 76.9)
- added R30: 3.3k, Resistor_SMD:R_0805_2012Metric, F.Cu at (103.6, 77.3)
- added R31: 3.3k, Resistor_SMD:R_0805_2012Metric, F.Cu at (106.3, 77.2)
- added R32: 3.3k, Resistor_SMD:R_0805_2012Metric, F.Cu at (108.9, 77.2)
- added R33: 3.3k, Resistor_SMD:R_0805_2012Metric, F.Cu at (111.3, 77.2)
- added R34: 3.3k, Resistor_SMD:R_0805_2012Metric, F.Cu at (113.8, 77.2)
- added R35: 3.3k, Resistor_SMD:R_0805_2012Metric, F.Cu at (116.6, 77.2)
- added R36: 3.3k, Resistor_SMD:R_0805_2012Metric, F.Cu at (119.1, 77.2)
- added R37: 3.3k, Resistor_SMD:R_0805_2012Metric, F.Cu at (121.7, 77.1)
- added R38: R, Resistor_SMD:R_0805_2012Metric, F.Cu at (108.3, 71.0)
- added R39: R, Resistor_SMD:R_0805_2012Metric, F.Cu at (105.4, 68.2)
- added R40: 3.3k, Resistor_SMD:R_0805_2012Metric, F.Cu at (119.0, 112.7)
- added R41: 3.3k, Resistor_SMD:R_0805_2012Metric, F.Cu at (93.2, 112.8)
- added R42: 3.3k, Resistor_SMD:R_0805_2012Metric, F.Cu at (116.4, 112.7)
- added R43: 3.3k, Resistor_SMD:R_0805_2012Metric, F.Cu at (90.6, 112.8)
- added R44: 3.3k, Resistor_SMD:R_0805_2012Metric, F.Cu at (113.8, 112.7)
- added R45: 3.3k, Resistor_SMD:R_0805_2012Metric, F.Cu at (88.0, 112.8)
- added R46: 3.3k, Resistor_SMD:R_0805_2012Metric, F.Cu at (111.2, 112.7)
- added R47: 3.3k, Resistor_SMD:R_0805_2012Metric, F.Cu at (85.6, 112.8)
- added R48: 3.3k, Resistor_SMD:R_0805_2012Metric, F.Cu at (108.8, 112.7)
- added R49: 3.3k, Resistor_SMD:R_0805_2012Metric, F.Cu at (83.0, 112.8)
- added R50: 3.3k, Resistor_SMD:R_0805_2012Metric, F.Cu at (106.0, 112.7)
- added R51: 3.3k, Resistor_SMD:R_0805_2012Metric, F.Cu at (80.4, 112.8)
- added R52: 3.3k, Resistor_SMD:R_0805_2012Metric, F.Cu at (103.2, 112.7)
- added R53: 3.3k, Resistor_SMD:R_0805_2012Metric, F.Cu at (78.0, 112.8)
- added R54: 3.3k, Resistor_SMD:R_0805_2012Metric, F.Cu at (101.0, 112.7)
- added R55: 3.3k, Resistor_SMD:R_0805_2012Metric, F.Cu at (75.4, 112.8)
- added R56: R, Resistor_SMD:R_0805_2012Metric, F.Cu at (118.8, 121.4)
- added R57: R, Resistor_SMD:R_0805_2012Metric, F.Cu at (92.0, 121.1)
- added R58: R, Resistor_SMD:R_0805_2012Metric, F.Cu at (117.8, 116.8)
- added R59: R, Resistor_SMD:R_0805_2012Metric, F.Cu at (91.0, 116.9)
- added R60: R, Resistor_SMD:R_0805_2012Metric, F.Cu at (122.4, 93.4)
- added R61: R, Resistor_SMD:R_0805_2012Metric, F.Cu at (102.8, 97.1)
- added TP1: FT_CLKOUT_TP, TestPoint:TestPoint_Pad_D1.5mm, F.Cu at (75.0, 89.8)
- added TP2: SDO, TestPoint:TestPoint_Pad_D1.5mm, F.Cu at (125.4, 93.8)
- added U5: SN74LVC8T245, Package_SO:TSSOP-24_4.4x7.8mm_P0.65mm, F.Cu at (88.1, 69.9)
- added U6: SN74LVC8T245, Package_SO:TSSOP-24_4.4x7.8mm_P0.65mm, F.Cu at (118.7, 70.1)
- added U7: SN74LVC8T245, Package_SO:TSSOP-24_4.4x7.8mm_P0.65mm, F.Cu at (106.7, 119.2)
- added U8: SN74LVC8T245, Package_SO:TSSOP-24_4.4x7.8mm_P0.65mm, F.Cu at (80.2, 119.3)
- added U9: ~, Package_DFN_QFN:UQFN-28-1EP_4x4mm_P0.4mm_EP2.35x2.35mm_ThermalVias, F.Cu at (114.9, 93.9)
- C15: value 0.1 uF -> C
- J2: value Conn_ARM_JTAG_SWD_10 -> TAnalog; footprint Connector_PinHeader_1.27mm:PinHeader_2x05_P1.27mm_Vertical_SMD -> Connector_PinHeader_2.54mm:PinHeader_1x02_P2.54mm_Vertical
- J3: value Conn_01x16 -> TDigital; footprint Connector_PinHeader_2.54mm:PinHeader_1x16_P2.54mm_Vertical -> Connector_PinHeader_2.54mm:PinHeader_1x02_P2.54mm_Vertical
- J4: value Conn_01x16 -> OUT_A; footprint Connector_PinHeader_2.54mm:PinHeader_1x16_P2.54mm_Vertical -> Connector_PinHeader_2.54mm:PinHeader_1x08_P2.54mm_Vertical
- J6, J7: value POWER -> 3v3
- moved J3 61.0 mm to (127.1, 111.6), turned to -90 degrees
- moved J4 58.8 mm to (75.4, 63.6), turned to 90 degrees
- moved J6 48.7 mm to (64.2, 62.1), turned to 0 degrees
- moved J7 48.1 mm to (69.0, 62.1), turned to 0 degrees
- moved D1 38.1 mm to (65.2, 68.8), turned to 90 degrees
- moved R7 35.9 mm to (65.2, 72.5), turned to -90 degrees
- moved R13 30.6 mm to (64.2, 107.6)
- moved J2 30.3 mm to (105.6, 91.2)
- moved J1 30.2 mm to (59.8, 115.1)
- moved C2 29.6 mm to (60.8, 108.4), turned to 0 degrees
- moved C5 29.5 mm to (62.0, 80.0), turned to 180 degrees
- moved U4 29.4 mm to (60.0, 72.1), turned to 90 degrees
- moved R12 28.8 mm to (63.0, 121.8), turned to 0 degrees
- moved Y1 26.3 mm to (60.8, 105.8), turned to 90 degrees
- moved L1 26.2 mm to (67.1, 105.2)
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Connections:
- net /fpga/SPI_CS renamed SPI_CS
- net /fpga/SPI_MISO renamed SPI_MISO
- net /fpga/SPI_MOSI renamed SPI_MOSI
- net /fpga/SPI_SCK renamed SPI_SCK
- J2 pad 1: +3.3V -> GND
- J2 pad 2: TMS -> TVcca
- J3 pad 1: /fpga/PT23A -> GND
- J3 pad 2: /fpga/PT23B -> TVcc
- J4 pad 1: /fpga/PR21B -> Net-(J4-Pin_1)
- J4 pad 2: /fpga/PR28A -> Net-(J4-Pin_2)
- U1 pad 20: Net-(J4-Pin_16) -> D7
- U1 pad 21: Net-(J4-Pin_15) -> D6
- U1 pad 22: Net-(J4-Pin_14) -> D5
- U1 pad 23: Net-(J4-Pin_13) -> D4
- U1 pad 24: Net-(J4-Pin_12) -> D3
- U1 pad 26: Net-(J4-Pin_11) -> D2
- U1 pad 27: Net-(J4-Pin_10) -> D1
- U1 pad 28: Net-(J4-Pin_9) -> D0
- U1 pad 30: Net-(J4-Pin_8) -> C7
- U1 pad 31: Net-(J4-Pin_7) -> C6
- U1 pad 33: Net-(J4-Pin_6) -> C5
- U1 pad 34: Net-(J4-Pin_5) -> C4
- U1 pad 35: Net-(J4-Pin_4) -> C3
- U1 pad 36: Net-(J4-Pin_3) -> C2
- U1 pad 37: /fpga/PR28A -> C1
- U1 pad 38: /fpga/PR21B -> C0
- U1 pad 4: FT_WR -> FT_CLKOUT
- U1 pad 45: Net-(J3-Pin_16) -> B7
- U1 pad 47: Net-(J3-Pin_15) -> B6
- U1 pad 49: Net-(J3-Pin_14) -> B5
- U1 pad 50: Net-(J3-Pin_13) -> B4
- U1 pad 51: Net-(J3-Pin_12) -> B3
- U1 pad 52: Net-(J3-Pin_11) -> B2
- U1 pad 53: Net-(J3-Pin_10) -> B1
- U1 pad 56: /fpga/PT39B -> B0
- U1 pad 57: /fpga/PT39A -> A7
- U1 pad 58: /fpga/PT38B -> A6
- U1 pad 59: /fpga/PT38A -> A5
- U1 pad 6: FT_RD -> FT_WR
- U1 pad 63: /fpga/PT28B -> A4
- U1 pad 65: /fpga/PT28A -> A3
- U1 pad 66: /fpga/PT27D/SDA/PCLKC0 -> A2
- U1 pad 67: OSC_12MHz -> Net-(D3-A)
- U1 pad 68: /fpga/PT23B -> A1
- U1 pad 69: /fpga/PT23A -> A0
- U1 pad 7: FT_TXE -> FT_RD
- U1 pad 8: FT_CLKOUT -> FT_TXE
- U2 pad 3: OSC_12MHz -> Net-(U2-OSCI)
- Y1 pad 3: OSC_12MHz -> Net-(U2-OSCI)
Routing:
- net TVcc: track 0.00 -> 216.4 mm
- net GND: track 106.0 -> 170.6 mm, vias 74 -> 125
- net OSC_12MHz: track 54.5 -> 0.00 mm
- net VBUS: track 14.7 -> 65.6 mm
- net C0: track 0.00 -> 49.3 mm
- net B7: track 0.00 -> 48.7 mm
- net C1: track 0.00 -> 44.6 mm
- net B6: track 0.00 -> 44.2 mm
- net B5: track 0.00 -> 40.4 mm
- net C2: track 0.00 -> 40.2 mm
- net B4: track 0.00 -> 39.8 mm
- net B3: track 0.00 -> 39.4 mm
- net B2: track 0.00 -> 38.8 mm
- net B1: track 0.00 -> 37.6 mm
- net B0: track 0.00 -> 37.2 mm
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Other:
- board size 78 x 34 mm -> 75 x 70 mm
- board text removed: "PB16A"
- board text removed: "PB18A"
- board text removed: "PB18B"
- board text removed: "PB22A"
- board text removed: "PB22B"
- board text removed: "PB29A"
- board text removed: "PB29B"
- board text removed: "PB32A"
- board text removed: "PB35A"
- board text removed: "PB35B"
- board text removed: "PB41A"
- board text removed: "PB41B"
- board text removed: "PB46A"
- board text removed: "PB46B"
- board text removed: "PR12A"
- board text removed: "PR21B"
- board text removed: "PR28A"
- board text removed: "PR2A"
- board text removed: "PR2B"
- board text removed: "PR2C"
- board text removed: "PR3A"
- board text removed: "PR3B"
- board text removed: "PR5A"
- board text removed: "PT28A"
- board text removed: "PT28B"
- board text removed: "PT38A"
- board text removed: "PT38B"
- board text removed: "PT39A"
- board text removed: "PT39B"

Commit message: finalize
Parts:
- moved R61 2.11 mm to (104.9, 97.3)
Connections:
- net Net-(U2-DM) renamed /D-
- net Net-(U2-DP) renamed /D+
Routing:
- net +3.3V: track 475.1 -> 478.5 mm
- net Net-(JP5-B): track 19.7 -> 18.0 mm
- net /D-: track 22.9 -> 24.4 mm
- net TVcca: track 27.9 -> 26.9 mm
- net GND: track 170.6 -> 169.6 mm
- net A3: track 21.7 -> 21.1 mm
Other:
- rule pad_to_mask_clearance: 0 -> 0.0508
- board text added: "+"
- board text added: "-"
- board text added: "3v"
- board text added: "5v"
- board text added: "A0"
- board text added: "A1"
- board text added: "A2"
- board text added: "A3"
- board text added: "A4"
- board text added: "A5"
- board text added: "A6"
- board text added: "A7"
- board text added: "AN0"
- board text added: "AN1"
- board text added: "AN10"
- board text added: "AN11"
- board text added: "AN12"
- board text added: "AN13"
- board text added: "AN14"
- board text added: "AN15"
- board text added: "AN2"
- board text added: "AN3"
- board text added: "AN4"
- board text added: "AN5"
- board text added: "AN6"
- board text added: "AN7"
- board text added: "AN8"
- board text added: "AN9"
- board text added: "ANLG PWR"
- board text added: "B0"
- board text added: "B1"
- board text added: "B2"
- board text added: "B3"
- board text added: "B4"
- board text added: "B5"
- board text added: "B6"
- board text added: "B7"
- board text added: "C0"
- board text added: "C1"
- board text added: "C2"
- board text added: "C3"
- board text added: "C4"
- board text added: "C5"
- board text added: "C6"
- board text added: "C7"
- board text added: "D0"
- board text added: "D1"
- board text added: "D2"
- board text added: "D3"
- board text added: "D4"
- board text added: "D5"
- board text added: "D6"
- board text added: "D7"
- board text added: "IN"
- board text added: "STATUS"
- board text added: "VBUS"
- board text added: "ViaEMS Test Bench V2"
- board text removed: "PT23A"
- board text removed: "PT23B"
- board text removed: "PT27D"
