File: test-harness/test-harness.kicad_sch (KiCad schematic)
At the start: 35 parts, among them J1 USB_C_Receptacle_USB2.0_16P, J6 POWER, J7 POWER, U2 FT2232H-56Q, U3 93CxxC, U4 TPS7B88Q1, Y1 12 MHz

Commit message: bump
Parts:
- D2: Digikey-Part (none) -> 478-7800-1-ND
- U2: Digikey-Part (none) -> 768-1276-ND
Changed lines of the file:
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@@
+			)
+		)
+		(property "Digikey-Part" "478-7800-1-ND"
+			(at 24.13 22.86 0)
+			(effects
+				(font
+					(size 1.27 1.27)
+				)
+				(hide yes)
 			)
 		)
@@
 			(at 135.89 114.3 0)
 			(effects
+				(font
+					(size 1.27 1.27)
+				)
+				(hide yes)
+			)
+		)
+		(property "Digikey-Part" " 768-1276-ND"
+			(at 135.89 114.3 0)
+			(effects
