File: test-harness/test-harness.kicad_sch (KiCad schematic)
At the start: 35 parts, among them J1 USB_C_Receptacle_USB2.0_16P, J6 POWER, J7 POWER, U2 FT2232H-56Q, U3 93CxxC, U4 TPS7B88Q1, Y1 12 MHz

Commit message: Test harness v2
Parts:
- added H1, H2, H3, H4: MountingHole, MountingHole:MountingHole_2.5mm_Pad, symbol Mechanical:MountingHole
- added J17, J8: 5v_usb, Connector_PinHeader_2.54mm:PinHeader_1x02_P2.54mm_Vertical, symbol Connector_Generic:Conn_01x02
- added J2: TAnalog, Connector_PinHeader_2.54mm:PinHeader_1x02_P2.54mm_Vertical, symbol Connector_Generic:Conn_01x02
- added J3: TDigital, Connector_PinHeader_2.54mm:PinHeader_1x02_P2.54mm_Vertical, symbol Connector_Generic:Conn_01x02
- added TP1: FT_CLKOUT_TP, TestPoint:TestPoint_Pad_D1.5mm, symbol Connector:TestPoint
- J6, J7: value POWER -> 3v3
Connections:
- net FT_CLKOUT: now also TP1.1
- net GND: now also J17.1 (Pin_1), J2.1 (Pin_1), J3.1 (Pin_1), J8.1 (Pin_1)
- net VBUS: now also J17.2 (Pin_2), J8.2 (Pin_2)
- net OSC_12MHz: no longer names the net of U2.3 (OSCI), Y1.3 (OUT)
- new net TVcc: J3.2 (Pin_2)
- new net TVcca: J2.2 (Pin_2)
Other:
- added sheet Analog (analog.kicad_sch)
- added sheet IO (io.kicad_sch)
- moved on the sheet: J6, J7

Commit message: finalize
Connections:
- net D+: now reaches J1.A6 (D+), J1.B6 (D+), U2.8 (DP)
- net D-: now reaches J1.A7 (D-), J1.B7 (D-), U2.7 (DM)
Changed lines of the file:
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@@
+		)
+	)
+	(label "D+"
+		(at 83.82 90.17 0)
+		(effects
+			(font
+				(size 1.27 1.27)
+			)
+			(justify left bottom)
+		)
+	)
+	(label "D-"
+		(at 88.9 90.17 0)
+		(effects
+			(font
+				(size 1.27 1.27)
+			)
+			(justify left bottom)
 		)
 	)
